File: VESC6_OPEN_HARDWARE.kicad_pcb (KiCad board)
At the start: 4 copper layers, 110 x 45 mm, 131 parts, among them P10 PH_A, P11 SUPPLY, P12 GND, P8 PH_C, P9 PH_B, Q1 STL130N6F7, Q2 STL130N6F7, Q3 STL130N6F7, Q4 STL130N6F7, Q5 STL130N6F7, Q6 STL130N6F7, U1 STM32F40X_LQFP64, U10 LSM6DS3TR-C, U2 LM3671, U3 DRV8301, U4 TJA1051TK-3, U5 AD8418, U6 AD8418, U7 AD8418, X1 8m

Commit message: prep for chaneling. fixed the connector references, added cha to this schematic.
Parts:
- removed USB: USB_OTG, Connector_USB:USB_Micro-B_Molex_47346-0001
- added J1: USB_C_Receptacle_USB2.0_16P, Connector_USB:USB_C_Receptacle_HRO_TYPE-C-31-M-12, F.Cu at (76.7, -13.9)
- added R4: 5k1, Resistor_SMD:R_0805_2012Metric_Pad1.20x1.40mm_HandSolder, F.Cu at (72.7, -6.10)
- added R5: 5k1, Resistor_SMD:R_0805_2012Metric_Pad1.20x1.40mm_HandSolder, F.Cu at (80.7, -6.10)
- added U8: USBLC6-2SC6, Package_TO_SOT_SMD:SOT-23-6, F.Cu at (76.7, -5.90)
- P2: renamed from CAN; value CAN1 -> CAN 1
- P5: renamed from CAN; value CAN2 -> CAN 2
- renumbered SWD to P3, SENSE to P4, ADC/SW to P6
Connections:
- net +5V renamed +5VA
- net VCC renamed +3V3a
- P2 pad MP: (no net) -> GND
- P3 pad MP: (no net) -> GND
- P4 pad MP: (no net) -> GND
- P5 pad MP: (no net) -> GND
- P6 pad MP: (no net) -> GND
- R1 pad 2: Net-(P1-VBUS) -> /USB/VBUS
- R2 pad 2: Net-(P1-D-) -> /USB/USB_D-
- R3 pad 2: Net-(P1-D+) -> /USB/USB_D+
Routing:
- net /USB/VBUS: track 0.00 -> 28.5 mm, vias 0 -> 4
- net Net-(P1-VBUS): track 18.2 -> 0.00 mm, vias 2 -> 0
- net /USB/D+: track 0.00 -> 11.1 mm
- net /USB/D-: track 0.00 -> 8.03 mm, vias 0 -> 2
- net /USB/CC1: track 0.00 -> 6.48 mm
- net /USB/CC2: track 0.00 -> 6.27 mm
- net Net-(P1-D-): track 6.07 -> 0.00 mm
- net /USB/USB_D-: track 0.00 -> 6.07 mm
- net Net-(P1-D+): track 5.16 -> 0.00 mm
- net /USB/USB_D+: track 0.00 -> 5.16 mm
- net GND: vias 203 -> 204
Other:
- outline, holes or cut-outs redrawn

Commit message: more fixes for channels
Parts:
- renumbered C58 to C1001, C61 to C1002, C62 to C1003, C33 to C1004, C34 to C1005, C2 to C1006, C3 to C1007, C4 to C1008, C7 to C1009, C5 to C1010, C6 to C1011, C8 to C1012, C9 to C1013, C10 to C1014, C11 to C1015, C12 to C1016, C13 to C1017, C14 to C1018, C15 to C1019, C17 to C1020, C16 to C1021, C20 to C1022, C18 to C1023, C19 to C1024, C64 to C1025, C21 to C1026, C22 to C1027, C26 to C1028, C23 to C1029, C24 to C1030, C25 to C1031, C28 to C1032, C27 to C1033, C31 to C1034, C32 to C1035, C35 to C1036, C29 to C1037, C30 to C1038, C45 to C1039, C37 to C1040, C39 to C1041, C38 to C1042, C36 to C1043, C40 to C1044, C41 to C1045, C42 to C1046, C43 to C1051, C44 to C1052, D2 to D1001, D3 to D1002, D4 to D1003, D5 to D1004, H1 to H1001, H2 to H1002, H3 to H1003, H4 to H1004, J1 to J1001, L1 to L1001, L2 to L1002, P5 to P1001, P3 to P1002, P2 to P1003, P4 to P1004, P6 to P1005, P8 to P1006, P9 to P1007, P10 to P1008, Q1 to Q1001, Q2 to Q1002, Q3 to Q1003, Q4 to Q1004, Q5 to Q1005, Q6 to Q1006, R42 to R1001, R43 to R1002, R44 to R1003, R1 to R1004, R2 to R1005, R3 to R1006, R39 to R1007, R8 to R1008, R9 to R1009, R40 to R1010, R41 to R1011, R23 to R1012, R10 to R1013, R11 to R1014, R12 to R1015, R13 to R1016, R14 to R1017, R38 to R1018, R15 to R1019, R16 to R1020, R17 to R1021, R18 to R1022, R19 to R1023, R20 to R1024, R21 to R1025, R22 to R1026, R4 to R1027, R5 to R1028, R24 to R1029, R25 to R1030, R26 to R1031, R35 to R1032, R36 to R1033, R37 to R1034, R29 to R1035, R27 to R1036, R28 to R1037, R30 to R1038, R31 to R1039, R32 to R1040, R33 to R1041, R34 to R1042, U10 to U1001, U4 to U1002, U1 to U1003, U2 to U1004, U3 to U1005, U8 to U1006, U5 to U1007, U6 to U1008, U7 to U1009, X1 to X1001
Connections:
- net +5VA renamed +5Va
- net /CAN/CANH renamed /CHa/CAN/CANH
- net /CAN/CANL renamed /CHa/CAN/CANL
- net /CAN/RX renamed /CHa/CAN/RX
- net /CAN/TX renamed /CHa/CAN/TX
- net /DRV8301/CS renamed /CHa/DRV8301/CS
- net /DRV8301/EN_GATE renamed /CHa/DRV8301/EN_GATE
- net /DRV8301/FAULT renamed /CHa/DRV8301/FAULT
- net /DRV8301/GH_A renamed /CHa/DRV8301/GH_A
- net /DRV8301/GH_B renamed /CHa/DRV8301/GH_B
- net /DRV8301/GH_C renamed /CHa/DRV8301/GH_C
- net /DRV8301/GL_A renamed /CHa/DRV8301/GL_A
- net /DRV8301/GL_B renamed /CHa/DRV8301/GL_B
- net /DRV8301/GL_C renamed /CHa/DRV8301/GL_C
- net /DRV8301/INH_A renamed /CHa/DRV8301/INH_A
- net /DRV8301/INH_B renamed /CHa/DRV8301/INH_B
- net /DRV8301/INH_C renamed /CHa/DRV8301/INH_C
- net /DRV8301/INL_A renamed /CHa/DRV8301/INL_A
- net /DRV8301/INL_B renamed /CHa/DRV8301/INL_B
- net /DRV8301/INL_C renamed /CHa/DRV8301/INL_C
- net /DRV8301/SCLK renamed /CHa/DRV8301/SCLK
- net /DRV8301/SDI renamed /CHa/DRV8301/SDI
- net /DRV8301/SDO renamed /CHa/DRV8301/SDO
- net /DRV8301/SENS_A renamed /CHa/DRV8301/SENS_A
- net /DRV8301/SENS_B renamed /CHa/DRV8301/SENS_B
- net /DRV8301/SENS_C renamed /CHa/DRV8301/SENS_C
- net /DRV8301/SENS_SUPPLY renamed /CHa/DRV8301/SENS_SUPPLY
- net /DRV8301/SH_A renamed /CHa/DRV8301/SH_A
- net /DRV8301/SH_B renamed /CHa/DRV8301/SH_B
- net /DRV8301/SH_C renamed /CHa/DRV8301/SH_C
- net /DRV8301/SWITCH- renamed /CHa/DRV8301/SWITCH-
- net /IMU/SCL renamed /CHa/IMU/SCL
- net /IMU/SDA renamed /CHa/IMU/SDA
- net /USB/CC1 renamed /CHa/USB/CC1
- net /USB/CC2 renamed /CHa/USB/CC2
- net /USB/D+ renamed /CHa/USB/D+
- net /USB/D- renamed /CHa/USB/D-
- net /USB/USB_D+ renamed /CHa/USB/USB_D+
- net /USB/USB_D- renamed /CHa/USB/USB_D-
- net /USB/VBUS renamed /CHa/USB/VBUS
- net /power/CURR_A renamed /CHa/Hbridge/CURR_A
- net /power/CURR_B renamed /CHa/Hbridge/CURR_B
- net /power/CURR_C renamed /CHa/Hbridge/CURR_C
- net /power/C_A renamed /CHa/Hbridge/C_A
- net /power/C_B renamed /CHa/Hbridge/C_B
- net /power/C_C renamed /CHa/Hbridge/C_C
- net /power/TEMP renamed /CHa/Hbridge/TEMP
- net /stm32f40x/ADC_15 renamed /CHa/stm32f40x/ADC_15
- net /stm32f40x/HALL_1 renamed /CHa/stm32f40x/HALL_1
- net /stm32f40x/HALL_2 renamed /CHa/stm32f40x/HALL_2
- net /stm32f40x/HALL_3 renamed /CHa/stm32f40x/HALL_3
- net /stm32f40x/LED_GREEN renamed /CHa/stm32f40x/LED_GREEN
- net /stm32f40x/LED_RED renamed /CHa/stm32f40x/LED_RED
- net /stm32f40x/MISO_ADC_EXT2 renamed /CHa/stm32f40x/MISO_ADC_EXT2
- net /stm32f40x/NRST renamed /CHa/stm32f40x/NRST
- net /stm32f40x/PB12 renamed /CHa/stm32f40x/PB12
- net /stm32f40x/PB3 renamed /CHa/stm32f40x/PB3
- net /stm32f40x/PB4 renamed /CHa/stm32f40x/PB4
- net /stm32f40x/PD2 renamed /CHa/stm32f40x/PD2
- net /stm32f40x/RX_SDA_NSS renamed /CHa/stm32f40x/RX_SDA_NSS
- net /stm32f40x/SCK_ADC_EXT renamed /CHa/stm32f40x/SCK_ADC_EXT
- net /stm32f40x/SERVO renamed /CHa/stm32f40x/SERVO
- net /stm32f40x/SWCLK renamed /CHa/stm32f40x/SWCLK
- net /stm32f40x/SWDIO renamed /CHa/stm32f40x/SWDIO
- net /stm32f40x/TEMP_MOTOR renamed /CHa/stm32f40x/TEMP_MOTOR
- net /stm32f40x/TX_SCL_MOSI renamed /CHa/stm32f40x/TX_SCL_MOSI
- net /stm32f40x/USB_DM renamed /CHa/stm32f40x/USB_DM
- net /stm32f40x/USB_DP renamed /CHa/stm32f40x/USB_DP

Commit message: relinked UUIDs
Parts:
- renumbered C51 to C1, C1004 to C101, C1005 to C102, C1017 to C103, C1018 to C104, C1019 to C105, C1020 to C106, C1021 to C107, C1022 to C108, C1023 to C109, C1024 to C110, C1025 to C111, C1026 to C112, C1027 to C113, C1028 to C114, C1029 to C115, C1030 to C116, C1031 to C117, C1032 to C118, C1033 to C119, C1034 to C120, C1035 to C121, C1036 to C122, C1037 to C123, C1038 to C124, C1039 to C125, C1040 to C126, C1041 to C127, C1042 to C128, C1043 to C129, C1044 to C130, C1045 to C131, C1046 to C132, C1051 to C133, C1052 to C134, C1002 to C135, C1003 to C136, C1006 to C137, C1007 to C138, C1008 to C139, C1009 to C140, C1010 to C141, C1011 to C142, C1012 to C143, C1013 to C144, C1014 to C145, C1015 to C146, C1016 to C147, C1001 to C148, C50 to C2, C48 to C3, C49 to C4, D1003 to D101, D1004 to D102, D1001 to D103, D1002 to D104, J1001 to J101, L1001 to L101, L1002 to L102, P11 to P1, P1006 to P101, P1007 to P102, P1008 to P103, P1001 to P104, P1003 to P105, P1002 to P106, P1004 to P107, P1005 to P108, P12 to P2, Q1001 to Q101, Q1002 to Q102, Q1003 to Q103, Q1004 to Q104, Q1005 to Q105, Q1006 to Q106, R1012 to R101, R1013 to R102, R1014 to R103, R1015 to R104, R1016 to R105, R1017 to R106, R1018 to R107, R1019 to R108, R1020 to R109, R1021 to R110, R1022 to R111, R1023 to R112, R1024 to R113, R1025 to R114, R1026 to R115, R1029 to R116, R1030 to R117, R1031 to R118, R1032 to R119, R1033 to R120, R1034 to R121, R1035 to R122, R1036 to R123, R1037 to R124, R1038 to R125, R1039 to R126, R1040 to R127, R1041 to R128, R1042 to R129, R1010 to R130, R1011 to R131, R1027 to R132, R1028 to R133, R1001 to R134, R1002 to R135, R1003 to R136, R1004 to R137, R1005 to R138, R1006 to R139, R1007 to R140, R1008 to R141, R1009 to R142, U1002 to U101, U1004 to U102, U1005 to U103, U1007 to U104, U1008 to U105, U1009 to U106, U1001 to U107, U1006 to U108, U1003 to U109, X1001 to X101
