File: VESC6_OPEN_HARDWARE.kicad_pcb (KiCad board)
At the start: 4 copper layers, 110 x 45 mm, 134 parts, among them J101 USB_C_Receptacle_USB2.0_16P, P1 SUPPLY, P101 PH_C, P102 PH_B, P103 PH_A, P104 CAN 2, P105 CAN 1, P106 SWD, P107 HALL/Encoder, P108 ADC_SWITCH, P2 GND, Q101 STL130N6F7, Q102 STL130N6F7, Q103 STL130N6F7, Q104 STL130N6F7, Q105 STL130N6F7, Q106 STL130N6F7, U101 TJA1051TK-3, U102 LM3671, U103 DRV8301, U104 AD8418, U105 AD8418, U106 AD8418, U107 LSM6DS3TR-C, U108 USBLC6-2SC6, U109 STM32F40X_LQFP64, X101 8m

Commit message: it seems to work. yay
Parts:
- renumbered H1001 to H1, H1002 to H2, H1003 to H3, H1004 to H4

Commit message: it looks like it's going together well!!!
Parts:
- added C2001: 2.2uF, Capacitor_SMD:C_0603_1608Metric, F.Cu at (70.6, 73.9)
- added C2002: 2.2uF, Capacitor_SMD:C_0603_1608Metric, F.Cu at (67.5, 73.9)
- added C2101: 2.2uF, Capacitor_SMD:C_0603_1608Metric, F.Cu at (76.4, 82.4)
- added C2102: 2.2uF, Capacitor_SMD:C_0603_1608Metric, F.Cu at (70.1, 65.8)
- added C2103: 2.2uF, Capacitor_SMD:C_0603_1608Metric, F.Cu at (68.6, 65.8)
- added C2104: 2.2uF, Capacitor_SMD:C_0603_1608Metric, F.Cu at (64.0, 59.6)
- added C2105: 6.8n, Capacitor_SMD:C_0603_1608Metric, F.Cu at (61.6, 79.5)
- added C2106: 2.2uF, Capacitor_SMD:C_0603_1608Metric, F.Cu at (64.0, 58.0)
- added C2107: 120p, Capacitor_SMD:C_0603_1608Metric, F.Cu at (62.0, 73.3)
- added C2108: 22n, Capacitor_SMD:C_0603_1608Metric, F.Cu at (67.1, 65.5)
- added C2109: 2.2uF, Capacitor_SMD:C_0603_1608Metric, F.Cu at (74.6, 79.4)
- added C2110: 100u, Capacitor_SMD:C_1210_3225Metric, F.Cu at (71.4, 79.3)
- added C2111: 15n, Capacitor_SMD:C_0603_1608Metric, F.Cu at (53.5, 74.0)
- added C2112: 4.7u_100v, Capacitor_SMD:C_1210_3225Metric, F.Cu at (51.1, 58.7)
- added C2113: 220n, Capacitor_SMD:C_0603_1608Metric, F.Cu at (51.2, 67.3)
- added C2114: 220n, Capacitor_SMD:C_0603_1608Metric, F.Cu at (51.2, 64.9)
- added C2115: 220n, Capacitor_SMD:C_0603_1608Metric, F.Cu at (51.2, 62.3)
- added C2116: 100n, Capacitor_SMD:C_0603_1608Metric, F.Cu at (51.2, 70.2)
- added C2117: 4.7u_100v, Capacitor_SMD:C_1210_3225Metric, F.Cu at (56.6, 74.1)
- added C2118: 2.2uF, Capacitor_SMD:C_0603_1608Metric, F.Cu at (58.2, 83.8)
- added C2119: 100u, Capacitor_SMD:C_1210_3225Metric, F.Cu at (61.7, 82.6)
- added C2201: 2.2uF, Capacitor_SMD:C_0603_1608Metric, F.Cu at (36.7, 56.8)
- added C2202: 4.7n, Capacitor_SMD:C_0603_1608Metric, F.Cu at (34.5, 77.4)
- added C2203: 4.7n, Capacitor_SMD:C_0603_1608Metric, F.Cu at (34.4, 67.5)
- added C2204: 4.7n, Capacitor_SMD:C_0603_1608Metric, F.Cu at (34.4, 57.5)
- added C2205: 4.7u_100v, Capacitor_SMD:C_1210_3225Metric, F.Cu at (34.8, 63.2)
- added C2206: 4.7u_100v, Capacitor_SMD:C_1210_3225Metric, F.Cu at (34.8, 59.9)
- added C2207: 2.2uF, Capacitor_SMD:C_0603_1608Metric, F.Cu at (36.7, 66.7)
- added C2208: 2.2uF, Capacitor_SMD:C_0603_1608Metric, F.Cu at (16.5, 85.8)
- added C2209: 4.7u_100v, Capacitor_SMD:C_1210_3225Metric, F.Cu at (34.8, 69.9)
- added C2210: 4.7u_100v, Capacitor_SMD:C_1210_3225Metric, F.Cu at (34.8, 73.2)
- added C2211: 2.2uF, Capacitor_SMD:C_0603_1608Metric, F.Cu at (36.8, 76.6)
- added C2212: 4.7u_100v, Capacitor_SMD:C_1210_3225Metric, F.Cu at (34.7, 83.1)
- added C2213: 4.7u_100v, Capacitor_SMD:C_1210_3225Metric, F.Cu at (34.7, 79.8)
- added C2301: 100n, Capacitor_SMD:C_0603_1608Metric, F.Cu at (86.4, 56.4)
- added C2302: 100n, Capacitor_SMD:C_0603_1608Metric, F.Cu at (91.9, 56.4)
- added C2501: 15p, Capacitor_SMD:C_0603_1608Metric, F.Cu at (78.3, 80.1)
- added C2502: 2.2uF, Capacitor_SMD:C_0603_1608Metric, F.Cu at (89.6, 63.6)
- added C2503: 2.2uF, Capacitor_SMD:C_0603_1608Metric, F.Cu at (75.0, 58.8)
- added C2504: 100n, Capacitor_SMD:C_0603_1608Metric, F.Cu at (72.9, 76.2)
- added C2505: 2.2uF, Capacitor_SMD:C_0603_1608Metric, F.Cu at (89.3, 72.9)
- added C2506: 2.2uF, Capacitor_SMD:C_0603_1608Metric, F.Cu at (90.9, 72.9)
- added C2507: 15p, Capacitor_SMD:C_0603_1608Metric, F.Cu at (81.5, 80.1)
- added C2508: 2.2uF, Capacitor_SMD:C_0603_1608Metric, F.Cu at (87.7, 72.9)
- added C2509: 2.2uF, Capacitor_SMD:C_0603_1608Metric, F.Cu at (72.0, 58.8)
- added C2510: 2.2uF, Capacitor_SMD:C_0603_1608Metric, F.Cu at (75.9, 76.2)
- added C2511: 2.2uF, Capacitor_SMD:C_0603_1608Metric, F.Cu at (92.7, 60.4)
- added C401: 100n, Capacitor_SMD:C_0603_1608Metric, F.Cu at (10.1, 53.5)
- added D2101: DIODE, Diode_SMD:D_SMF, F.Cu at (50.7, 73.5)
- added D2102: TVS 5V, Diode_SMD:D_SMA, F.Cu at (58.2, 79.4)
- added D401: RED, Diode_SMD:D_0603_1608Metric, F.Cu at (89.6, 65.2)
- added D402: WHITE, Diode_SMD:D_0603_1608Metric, F.Cu at (89.6, 66.8)
- added J2401: USB_C_Receptacle_USB2.0_16P, Connector_USB:USB_C_Receptacle_HRO_TYPE-C-31-M-12, F.Cu at (107.7, 52.6)
- added L2101: 2.2u, Inductor_SMD:L_0805_2012Metric, F.Cu at (70.0, 82.8)
- added L2102: 22u, Inductor_SMD:L_Taiyo-Yuden_NR-60xx_HandSoldering, F.Cu at (52.1, 80.2)
- added P2201: PH_C, Connector_Pin:Pin_D1.3mm_L11.0mm_LooseFit, F.Cu at (4.91, 60.5)
- added P2202: PH_B, Connector_Pin:Pin_D1.3mm_L11.0mm_LooseFit, F.Cu at (4.91, 70.5)
- added P2203: PH_A, Connector_Pin:Pin_D1.3mm_L11.0mm_LooseFit, F.Cu at (4.91, 80.5)
- added P401: CAN 2, Connector_JST:JST_SH_SM04B-SRSS-TB_1x04-1MP_P1.00mm_Horizontal, F.Cu at (36.4, 50.5)
- added P402: CAN 1, Connector_JST:JST_SH_SM04B-SRSS-TB_1x04-1MP_P1.00mm_Horizontal, F.Cu at (44.6, 50.5)
- added P403: SWD, Connector_JST:JST_SH_SM06B-SRSS-TB_1x06-1MP_P1.00mm_Horizontal, F.Cu at (53.8, 50.5)
- added P404: HALL/Encoder, Connector_JST:JST_SH_SM06B-SRSS-TB_1x06-1MP_P1.00mm_Horizontal, F.Cu at (3.37, 52.7)
- added P405: ADC_SWITCH, Connector_JST:JST_SH_SM04B-SRSS-TB_1x04-1MP_P1.00mm_Horizontal, F.Cu at (63.0, 50.5)
- added Q2201: STL130N6F7, CustomFootprints:NVMFS5C612NL, F.Cu at (28.6, 61.5)
- added Q2202: STL130N6F7, CustomFootprints:NVMFS5C612NL, F.Cu at (21.2, 59.5)
- added Q2203: STL130N6F7, CustomFootprints:NVMFS5C612NL, F.Cu at (28.6, 71.5)
- added Q2204: STL130N6F7, CustomFootprints:NVMFS5C612NL, F.Cu at (21.2, 69.6)
- added Q2205: STL130N6F7, CustomFootprints:NVMFS5C612NL, F.Cu at (28.5, 81.5)
- added Q2206: STL130N6F7, CustomFootprints:NVMFS5C612NL, F.Cu at (21.2, 79.5)
- added R2001: 120R, Resistor_SMD:R_0603_1608Metric, F.Cu at (68.2, 71.6)
- added R2101: 3.3k, Resistor_SMD:R_0603_1608Metric, F.Cu at (61.6, 77.9)
- added R2102: 18k, Resistor_SMD:R_0603_1608Metric, F.Cu at (61.6, 76.4)
- added R2103: 15k, Resistor_SMD:R_0603_1608Metric, F.Cu at (62.0, 74.8)
- added R2104: 10k, Resistor_SMD:R_0603_1608Metric, F.Cu at (63.9, 69.5)
- added R2105: 220k, Resistor_SMD:R_0603_1608Metric, F.Cu at (59.7, 74.0)
- added R2106: 10k, Resistor_SMD:R_0603_1608Metric, F.Cu at (68.0, 51.8)
- added R2107: 39k, Resistor_SMD:R_0603_1608Metric, F.Cu at (46.1, 83.8)
- added R2108: 2k2, Resistor_SMD:R_0603_1608Metric, F.Cu at (47.6, 82.0)
- added R2109: 39k, Resistor_SMD:R_0603_1608Metric, F.Cu at (39.0, 81.5)
- added R2110: 2k2, Resistor_SMD:R_0603_1608Metric, F.Cu at (42.1, 81.5)
- added R2111: 39k, Resistor_SMD:R_0603_1608Metric, F.Cu at (39.0, 71.6)
- added R2112: 2k2, Resistor_SMD:R_0603_1608Metric, F.Cu at (42.1, 71.6)
- added R2113: 39k, Resistor_SMD:R_0603_1608Metric, F.Cu at (39.1, 61.5)
- added R2114: 2k2, Resistor_SMD:R_0603_1608Metric, F.Cu at (42.1, 61.5)
- added R2201: 0.0005R, CustomFootprints:2512_SHUNT, F.Cu at (13.8, 60.5)
- added R2202: 4.7R, Resistor_SMD:R_0603_1608Metric, F.Cu at (16.1, 63.3)
- added R2203: 4.7R, Resistor_SMD:R_0603_1608Metric, F.Cu at (16.2, 56.4)
- added R2204: 100R, Resistor_SMD:R_0603_1608Metric, F.Cu at (34.5, 75.9)
- added R2205: 100R, Resistor_SMD:R_0603_1608Metric, F.Cu at (34.4, 66.0)
- added R2206: 100R, Resistor_SMD:R_0603_1608Metric, F.Cu at (34.4, 56.0)
- added R2207: 0.0005R, CustomFootprints:2512_SHUNT, F.Cu at (13.7, 70.5)
- added R2208: NTC 10k, Resistor_SMD:R_0603_1608Metric, F.Cu at (18.8, 86.6)
- added R2209: 10k, Resistor_SMD:R_0603_1608Metric, F.Cu at (16.5, 87.3)
- added R2210: 4.7R, Resistor_SMD:R_0603_1608Metric, F.Cu at (16.0, 73.4)
- added R2211: 4.7R, Resistor_SMD:R_0603_1608Metric, F.Cu at (16.1, 66.5)
- added R2212: 0.0005R, CustomFootprints:2512_SHUNT, F.Cu at (13.8, 80.5)
- added R2213: 4.7R, Resistor_SMD:R_0603_1608Metric, F.Cu at (16.1, 83.3)
- added R2214: 4.7R, Resistor_SMD:R_0603_1608Metric, F.Cu at (16.2, 76.4)
- added R2301: 1k, Resistor_SMD:R_0603_1608Metric, F.Cu at (88.8, 59.6)
- added R2302: 1k, Resistor_SMD:R_0603_1608Metric, F.Cu at (90.3, 59.6)
- added R2401: 5k1, Resistor_SMD:R_0805_2012Metric_Pad1.20x1.40mm_HandSolder, F.Cu at (99.9, 48.6)
- added R2402: 5k1, Resistor_SMD:R_0805_2012Metric_Pad1.20x1.40mm_HandSolder, F.Cu at (99.9, 56.6)
- added R401: 2k2, Resistor_SMD:R_0603_1608Metric, F.Cu at (10.1, 51.7)
- added R402: 2k2, Resistor_SMD:R_0603_1608Metric, F.Cu at (10.1, 50.1)
- added R403: 2k2, Resistor_SMD:R_0603_1608Metric, F.Cu at (10.1, 48.5)
- added R404: DNP, Resistor_SMD:R_0603_1608Metric, F.Cu at (69.7, 55.2)
- added R405: 22R, Resistor_SMD:R_0603_1608Metric, F.Cu at (78.8, 56.5)
- added R406: 22R, Resistor_SMD:R_0603_1608Metric, F.Cu at (77.3, 56.5)
- added R407: 10k, Resistor_SMD:R_0603_1608Metric, F.Cu at (13.1, 53.5)
- added R408: 120R, Resistor_SMD:R_0603_1608Metric, F.Cu at (92.4, 62.8)
- added R409: 120R, Resistor_SMD:R_0603_1608Metric, F.Cu at (92.7, 66.8)
- added U2001: TJA1051TK-3, Package_DFN_QFN:DFN-8-1EP_3x3mm_P0.65mm_EP1.55x2.4mm, F.Cu at (71.2, 71.3)
- added U2101: LM3671, Package_TO_SOT_SMD:SOT-23-5, F.Cu at (73.1, 82.7)
- added U2102: DRV8301, Package_SO:HTSSOP-56-1EP_6.1x14mm_P0.5mm_EP3.61x6.35mm, F.Cu at (57.6, 65.1)
- added U2201: AD8418, Package_SO:SOIC-8_3.9x4.9mm_P1.27mm, F.Cu at (41.3, 58.0)
- added U2202: AD8418, Package_SO:SOIC-8_3.9x4.9mm_P1.27mm, F.Cu at (41.3, 68.1)
- added U2203: AD8418, Package_SO:SOIC-8_3.9x4.9mm_P1.27mm, F.Cu at (41.3, 78.0)
- added U2301: LSM6DS3TR-C, Package_LGA:Bosch_LGA-14_3x2.5mm_P0.5mm, F.Cu at (89.2, 56.5)
- added U2401: USBLC6-2SC6, Package_TO_SOT_SMD:SOT-23-6, F.Cu at (99.7, 52.6)
- added U2501: STM32F40X_LQFP64, Package_QFP:LQFP-64_10x10mm_P0.5mm, F.Cu at (81.3, 67.0)
- added X2501: 8m, Crystal:Crystal_SMD_5032-2Pin_5.0x3.2mm, F.Cu at (79.9, 77.4)
- moved H102 100.0 mm to (85.0, 142.0)
- moved H103 100.0 mm to (25.0, 142.0)
- moved J1401 36.7 mm to (107.8, 5.60), turned to 90 degrees
- moved R1401 28.4 mm to (100.0, 1.60), turned to 0 degrees
- moved C201 26.8 mm to (122.5, 20.5)
- moved C202 26.8 mm to (122.5, 31.8)
- moved C203 26.8 mm to (122.5, 43.0)
- moved C204 26.8 mm to (122.5, 54.2)
- moved P201 26.8 mm to (129.8, 48.7)
- moved P202 26.8 mm to (129.8, 26.2)
- moved U1401 25.8 mm to (99.8, 5.60), turned to 180 degrees
- moved R1402 24.9 mm to (100.0, 9.60), turned to 0 degrees
- renumbered C101 to C1001, C102 to C1002, C103 to C1101, C104 to C1102, C105 to C1103, C106 to C1104, C107 to C1105, C108 to C1106, C109 to C1107, C110 to C1108, C111 to C1109, C112 to C1110, C113 to C1111, C114 to C1112, C115 to C1113, C116 to C1114, C117 to C1115, C118 to C1116, C119 to C1117, C120 to C1118, C121 to C1119, C122 to C1201, C123 to C1202, C124 to C1203, C125 to C1204, C126 to C1205, C127 to C1206, C128 to C1207, C129 to C1208, C130 to C1209, C131 to C1210, C132 to C1211, C133 to C1212, C134 to C1213, C135 to C1301, C136 to C1302, C137 to C1501, C138 to C1502, C139 to C1503, C140 to C1504, C141 to C1505, C142 to C1506, C143 to C1507, C144 to C1508, C145 to C1509, C146 to C1510, C147 to C1511, C1 to C201, C2 to C202, C3 to C203, C4 to C204, C148 to C301, D101 to D1101, D102 to D1102, D103 to D301, D104 to D302, H1 to H101, H2 to H102, H3 to H103, H4 to H104, J101 to J1401, L101 to L1101, L102 to L1102, P101 to P1201, P102 to P1202, P103 to P1203, P1 to P201, P2 to P202, P104 to P301, P105 to P302, P106 to P303, P107 to P304, P108 to P305, Q101 to Q1201, Q102 to Q1202, Q103 to Q1203, Q104 to Q1204, Q105 to Q1205, Q106 to Q1206, R101 to R1001, R102 to R1101, R103 to R1102, R104 to R1103, R105 to R1104, R106 to R1105, R107 to R1106, R108 to R1107, R109 to R1108, R110 to R1109, R111 to R1110, R112 to R1111, R113 to R1112, R114 to R1113, R115 to R1114, R116 to R1201, R117 to R1202, R118 to R1203, R119 to R1204, R120 to R1205, R121 to R1206, R122 to R1207, R123 to R1208, R124 to R1209, R125 to R1210, R126 to R1211, R127 to R1212, R128 to R1213, R129 to R1214, R130 to R1301, R131 to R1302, R132 to R1401, R133 to R1402, R134 to R301, R135 to R302, R136 to R303, R137 to R304, R138 to R305, R139 to R306, R140 to R307, R141 to R308, R142 to R309, U101 to U1001, U102 to U1101, U103 to U1102, U104 to U1201, U105 to U1202, U106 to U1203, U107 to U1301, U108 to U1401, U109 to U1501, X101 to X1501
Routing:
- net +3V3b: track 0.00 -> 308.7 mm, vias 0 -> 11
- net +5Vb: track 0.00 -> 197.3 mm, vias 0 -> 5
- net /CHb/stm32f40x/TEMP_MOTOR: track 0.00 -> 104.5 mm, vias 0 -> 2
- net /CHb/DRV8301/SWITCH-: track 0.00 -> 89.6 mm, vias 0 -> 2
- net /CHb/stm32f40x/HALL_3: track 0.00 -> 87.9 mm, vias 0 -> 2
- net /CHb/stm32f40x/HALL_2: track 0.00 -> 87.5 mm, vias 0 -> 2
- net /CHb/stm32f40x/HALL_1: track 0.00 -> 86.5 mm, vias 0 -> 2
- net /CHb/Hbridge/TEMP: track 0.00 -> 85.3 mm, vias 0 -> 2
- net /CHb/stm32f40x/NRST: track 0.00 -> 76.3 mm, vias 0 -> 2
- net /CHb/Hbridge/CURR_C: track 0.00 -> 74.1 mm, vias 0 -> 2
- net /CHb/Hbridge/CURR_B: track 0.00 -> 64.2 mm, vias 0 -> 2
- net /CHb/Hbridge/CURR_A: track 0.00 -> 64.1 mm, vias 0 -> 2
- net /CHb/DRV8301/SENS_C: track 0.00 -> 62.3 mm, vias 0 -> 2
- net /CHb/DRV8301/SENS_B: track 0.00 -> 60.5 mm, vias 0 -> 2
- net /CHb/DRV8301/SH_A: track 0.00 -> 58.2 mm, vias 0 -> 2
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- added copper zone on F.Cu, net /CHb/DRV8301/SH_A
- added copper zone on F.Cu, net /CHb/DRV8301/SH_B
- added copper zone on F.Cu, net /CHb/DRV8301/SH_C
- added copper zone on F.Cu, net Net-(P2201-Pin_1)
- added copper zone on F.Cu, net Net-(P2202-Pin_1)
- added copper zone on F.Cu, net Net-(P2203-Pin_1)
Other:
- board size 110 x 45 mm -> 110 x 90 mm

Commit message: small improvements.
Parts:
- removed the P401 at (36.4, 50.5)
- added C205: 220u_63v, Capacitor_SMD:CP_Elec_10x10.5, F.Cu at (26.5, 47.8)
- added C206: 4.7u_100v, Capacitor_SMD:C_1210_3225Metric, F.Cu at (26.2, 40.0)
- added C207: 4.7u_100v, Capacitor_SMD:C_1210_3225Metric, F.Cu at (37.8, 50.2)
- added H105: MountingHole, CustomFootprints:MountingHole_3mm, F.Cu at (11.0, 45.0)
- P401: renamed from P402; footprint Connector_JST:JST_SH_SM04B-SRSS-TB_1x04-1MP_P1.00mm_Horizontal -> Connector_JST:JST_SH_BM04B-SRSS-TB_1x04-1MP_P1.00mm_Vertical
- P403: footprint Connector_JST:JST_SH_SM06B-SRSS-TB_1x06-1MP_P1.00mm_Horizontal -> Connector_JST:JST_SH_BM06B-SRSS-TB_1x06-1MP_P1.00mm_Vertical
- P405: footprint Connector_JST:JST_SH_SM04B-SRSS-TB_1x04-1MP_P1.00mm_Horizontal -> Connector_JST:JST_SH_BM04B-SRSS-TB_1x04-1MP_P1.00mm_Vertical
- moved H103 56.8 mm to (11.0, 87.0)
- moved H102 55.0 mm to (85.0, 87.0)
- moved G*** 52.2 mm to (96.0, 86.2)
- moved C203 29.9 mm to (92.8, 40.5)
- moved P202 27.5 mm to (107.5, 42.2)
- moved P201 26.3 mm to (107.5, 34.8)
- moved G*** 26.1 mm to (102.5, 38.2), turned to 90 degrees
- moved G*** 24.2 mm to (70.0, 48.5)
- moved C202 22.5 mm to (100.3, 28.0)
- moved C201 22.5 mm to (100.3, 17.0)
- moved C204 19.1 mm to (103.5, 52.2), turned to -90 degrees
- moved J2401 13.3 mm to (107.7, 65.9)
- moved R2401 13.3 mm to (99.9, 61.9)
- moved R2402 13.3 mm to (99.9, 69.9)
- moved U2401 13.3 mm to (99.7, 65.9)
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Connections:
- P301 pad 1: /CHa/CAN/CANL -> /CHa/CANL
- P301 pad 2: /CHa/CAN/CANH -> /CHa/CANH
- P302 pad 1: /CHa/CAN/CANL -> /CHa/CANL
- P302 pad 2: /CHa/CAN/CANH -> /CHa/CANH
- P401 pad 1: /CHb/CAN/CANL -> /CHa/CANL
- P401 pad 2: /CHb/CAN/CANH -> /CHa/CANH
- R1001 pad 1: /CHa/CAN/CANH -> /CHa/CANH
- R1001 pad 2: /CHa/CAN/CANL -> /CHa/CANL
- R2001 pad 1: /CHb/CAN/CANH -> /CHa/CANH
- R2001 pad 2: /CHb/CAN/CANL -> /CHa/CANL
- U1001 pad 6: /CHa/CAN/CANL -> /CHa/CANL
- U1001 pad 7: /CHa/CAN/CANH -> /CHa/CANH
- U2001 pad 6: /CHb/CAN/CANL -> /CHa/CANL
- U2001 pad 7: /CHb/CAN/CANH -> /CHa/CANH
Routing:
- net /CHa/CANH: track 0.00 -> 138.8 mm, vias 0 -> 6
- net /CHa/CANL: track 0.00 -> 134.7 mm, vias 0 -> 8
- net SUPPLY: track 87.5 -> 183.6 mm, vias 31 -> 42
- net /CHb/CAN/CANH: track 48.2 -> 0.00 mm, vias 2 -> 0
- net /CHa/CAN/CANH: track 48.2 -> 0.00 mm, vias 2 -> 0
- net /CHb/CAN/CANL: track 46.2 -> 0.00 mm, vias 4 -> 0
- net /CHa/CAN/CANL: track 46.2 -> 0.00 mm, vias 4 -> 0
- net /CHb/USB/USB_D+: track 23.0 -> 32.1 mm
- net +5Vb: track 197.3 -> 206.4 mm, vias 5 -> 7
- net /CHb/USB/USB_D-: track 23.0 -> 32.1 mm
- net /CHb/USB/VBUS: track 46.7 -> 51.3 mm
- net /CHb/stm32f40x/NRST: track 76.3 -> 73.0 mm
- net /CHb/stm32f40x/SWDIO: track 33.2 -> 30.6 mm
- net /CHb/Hbridge/CURR_C: track 74.1 -> 71.7 mm
- net /CHb/stm32f40x/SWCLK: track 32.7 -> 30.8 mm
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Other:
- board text added: "Channel A"
- board text added: "Channel B"
- board text added: "Designed by Craig Gault github.com/craigg96 2ch fork by Tomáš Kuchta"
- board text removed: "Designed by Craig Gault github.com/craigg96"
