File: VESC6_OPEN_HARDWARE.kicad_pcb (KiCad board)
At the start: 4 copper layers, 110 x 90 mm, 258 parts, among them J1401 USB_C_Receptacle_USB2.0_16P, J2401 USB_C_Receptacle_USB2.0_16P, P1201 PH_C, P1202 PH_B, P1203 PH_A, P201 SUPPLY, P202 GND, P2201 PH_C, P2202 PH_B, P2203 PH_A, P301 CAN 2, P302 CAN 1, P303 SWD, P304 HALL/Encoder, P305 ADC_SWITCH, P401 CAN 1, P403 SWD, P404 HALL/Encoder, P405 ADC_SWITCH, Q1201 STL130N6F7, Q1202 STL130N6F7, Q1203 STL130N6F7, Q1204 STL130N6F7, Q1205 STL130N6F7, Q1206 STL130N6F7, Q2201 STL130N6F7, Q2202 STL130N6F7, Q2203 STL130N6F7, Q2204 STL130N6F7, Q2205 STL130N6F7, Q2206 STL130N6F7, U1001 TJA1051TK-3, U1101 LM3671, U1102 DRV8301, U1201 AD8418, U1202 AD8418, U1203 AD8418, U1301 LSM6DS3TR-C, U1401 USBLC6-2SC6, U1501 STM32F40X_LQFP64, U2001 TJA1051TK-3, U2101 LM3671, U2102 DRV8301, U2201 AD8418, U2202 AD8418, U2203 AD8418, U2301 LSM6DS3TR-C, U2401 USBLC6-2SC6, U2501 STM32F40X_LQFP64, X1501 8m, X2501 8m

Commit message: more fixes
Routing:
- net SUPPLY: vias 42 -> 93
- net GND: vias 452 -> 456
