File: USB.kicad_sch (KiCad schematic)
At the start: 4 parts, among them J1401 USB_C_Receptacle_USB2.0_16P, U1401 USBLC6-2SC6

Commit message: finishing touches
Parts:
- J1401: LCSC (none) -> C165948; LCSC part no. C165948 -> (none)
- R1401, R1402: LCSC (none) -> C84375; LCSC part no. C84375 -> (none)
- U1401: LCSC (none) -> C2827654; LCSC part no. C2827654 -> (none)
Changed lines of the file:
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@@
 			)
 		)
-		(property "LCSC" ""
-			(at 163.83 87.63 0)
-			(hide yes)
-			(show_name no)
-			(do_not_autoplace no)
-			(effects
-				(font
-					(size 1.27 1.27)
-				)
-			)
-		)
-		(property "LCSC part no." "C2827654"
+		(property "LCSC" "C2827654"
 			(at 163.83 87.63 0)
 			(hide yes)
@@
 			)
 		)
-		(property "LCSC" ""
-			(at 149.86 107.95 0)
-			(hide yes)
-			(show_name no)
-			(do_not_autoplace no)
-			(effects
-				(font
-					(size 1.27 1.27)
-				)
-			)
-		)
-		(property "LCSC part no." "C84375"
+		(property "LCSC" "C84375"
 			(at 149.86 107.95 0)
 			(hide yes)
@@
 			)
 		)
-		(property "LCSC" ""
-			(at 121.92 87.63 0)
-			(hide yes)
-			(show_name no)
-			(do_not_autoplace no)
-			(effects
-				(font
-					(size 1.27 1.27)
-				)
-			)
-		)
-		(property "LCSC part no." "C165948"
+		(property "LCSC" "C165948"
 			(at 121.92 87.63 0)
 			(hide yes)
@@
 			)
 		)
-		(property "LCSC" ""
+		(property "LCSC" "C84375"
 			(at 144.78 107.95 0)
 			(hide yes)
-			(show_name no)
-			(do_not_autoplace no)
-			(effects
-				(font
-					(size 1.27 1.27)
-				)
-			)
-		)
-		(property "LCSC part no." "C84375"
-			(at 144.78 107.95 0)
-			(hide yes)

Commit message: small improvements.
Parts:
- J1401: LCSC C165948 -> (none); LCSC part no. (none) -> C165948
- R1401, R1402: LCSC C84375 -> (none); LCSC part no. (none) -> C84375
- U1401: LCSC C2827654 -> (none); LCSC part no. (none) -> C2827654
Changed lines of the file:
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@@
 			)
 		)
-		(property "LCSC" "C2827654"
+		(property "LCSC" ""
+			(at 163.83 87.63 0)
+			(hide yes)
+			(show_name no)
+			(do_not_autoplace no)
+			(effects
+				(font
+					(size 1.27 1.27)
+				)
+			)
+		)
+		(property "LCSC part no." "C2827654"
 			(at 163.83 87.63 0)
 			(hide yes)
@@
 			)
 		)
-		(property "LCSC" "C84375"
+		(property "LCSC" ""
+			(at 149.86 107.95 0)
+			(hide yes)
+			(show_name no)
+			(do_not_autoplace no)
+			(effects
+				(font
+					(size 1.27 1.27)
+				)
+			)
+		)
+		(property "LCSC part no." "C84375"
 			(at 149.86 107.95 0)
 			(hide yes)
@@
 			)
 		)
-		(property "LCSC" "C165948"
+		(property "LCSC" ""
+			(at 121.92 87.63 0)
+			(hide yes)
+			(show_name no)
+			(do_not_autoplace no)
+			(effects
+				(font
+					(size 1.27 1.27)
+				)
+			)
+		)
+		(property "LCSC part no." "C165948"
 			(at 121.92 87.63 0)
 			(hide yes)
@@
 			)
 		)
-		(property "LCSC" "C84375"
+		(property "LCSC" ""
 			(at 144.78 107.95 0)
 			(hide yes)
+			(show_name no)
+			(do_not_autoplace no)
+			(effects
+				(font
+					(size 1.27 1.27)
+				)
+			)
+		)
+		(property "LCSC part no." "C84375"
+			(at 144.78 107.95 0)
+			(hide yes)
