File: CAN.kicad_sch (KiCad schematic)
At the start: 4 parts, among them U4 TJA1051TK-3

Commit message: prep for chaneling. fixed the connector references, added cha to this schematic.
Connections:
- net +5V renamed +5VA
- net VCC renamed +3V3a
Changed lines of the file:
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@@
 			)
 		)
-		(property "Value" "+5V"
+		(property "Value" "+5VA"
 			(at 117.221 69.2658 0)
 			(show_name no)
@@
 			)
 		)
-		(property "Value" "VCC"
+		(property "Value" "+3V3a"
 			(at 166.8018 69.2658 0)
 			(show_name no)

Commit message: more fixes for channels
Parts:
- renumbered C33 to C1004, C34 to C1005, R23 to R1012, U4 to U1002
Connections:
- net +3V3a renamed +3V3
- net +5VA renamed +5V
Changed lines of the file:
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@@
 	(wire
 		(pts
-			(xy 166.37 85.09) (xy 166.37 73.66)
+			(xy 166.37 72.39) (xy 166.37 85.09)
 		)
 		(stroke
@@
 			(width 0)
 			(type default)
+		)
+	)
+	(label "+5V"
+		(at 116.84 73.66 270)
+		(effects
+			(font
+				(size 1.27 1.27)
+			)
+			(justify right bottom)
+		)
+	)
+	(label "+3V3"
+		(at 166.37 72.39 270)
+		(effects
+			(font
+				(size 1.27 1.27)
+			)
+			(justify right bottom)
 		)
 	)
@@
 		)
 	)
+	(hierarchical_label "+5V"
+		(shape input)
+		(at 116.84 73.66 90)
+		(effects
+			(font
+				(size 1.27 1.27)
+			)
+			(justify left)
+		)
+	)
 	(hierarchical_label "TX"
 		(shape input)
@@
 			)
 			(justify right)
+		)
+	)
+	(hierarchical_label "+3V3"
+		(shape input)
+		(at 166.37 72.39 90)
+		(effects
+			(font
+				(size 1.27 1.27)
+			)
+			(justify left)
 		)
 	)
@@
 		(in_pos_files yes)
 		(dnp no)
-		(property "Reference" "C33"
+		(property "Reference" "C1004"
 			(at 118.11 87.63 0)
 			(show_name no)
@@
 		(instances
 			(project "VESC6_OPEN_HARDWARE"
-				(path "/8bc2c25a-a1f1-4ce8-b96a-a4f8f4c35079/00000000-0000-0000-0000-00005aeaa308"
-					(reference "C33")
+				(path "/8bc2c25a-a1f1-4ce8-b96a-a4f8f4c35079/1e81ec4a-7813-42c9-8244-ecd5bd9e7dba/b2b9706e-bd8f-4858-b41c-0ad60782e278"
+					(reference "C1004")
 					(unit 1)
 				)
@@
 		(in_pos_files yes)
 		(dnp no)
-		(property "Reference" "C34"
+		(property "Reference" "C1005"
 			(at 168.91 88.9 0)
 			(show_name no)
@@
 		(instances
 			(project "VESC6_OPEN_HARDWARE"
-				(path "/8bc2c25a-a1f1-4ce8-b96a-a4f8f4c35079/00000000-0000-0000-0000-00005aeaa308"
-					(reference "C34")
+				(path "/8bc2c25a-a1f1-4ce8-b96a-a4f8f4c35079/1e81ec4a-7813-42c9-8244-ecd5bd9e7dba/b2b9706e-bd8f-4858-b41c-0ad60782e278"
+					(reference "C1005")
 					(unit 1)
 				)
@@
 		(in_pos_files yes)
 		(dnp no)
-		(property "Reference" "R23"
+		(property "Reference" "R1012"
 			(at 181.61 82.55 90)
 			(show_name no)
@@
 		(instances
 			(project "VESC6_OPEN_HARDWARE"
-				(path "/8bc2c25a-a1f1-4ce8-b96a-a4f8f4c35079/00000000-0000-0000-0000-00005aeaa308"
-					(reference "R23")
+				(path "/8bc2c25a-a1f1-4ce8-b96a-a4f8f4c35079/1e81ec4a-7813-42c9-8244-ecd5bd9e7dba/b2b9706e-bd8f-4858-b41c-0ad60782e278"
+					(reference "R1012")
 					(unit 1)
 				)
@@
 		(in_pos_files yes)
 		(dnp no)
-		(property "Reference" "U4"
+		(property "Reference" "U1002"
 			(at 145.415 70.739 0)
 			(show_name no)
@@
 		(instances
 			(project "VESC6_OPEN_HARDWARE"
-				(path "/8bc2c25a-a1f1-4ce8-b96a-a4f8f4c35079/00000000-0000-0000-0000-00005aeaa308"
-					(reference "U4")
-					(unit 1)
-				)
-			)
-		)
-	)
-	(symbol
-		(lib_id "power:+5V")
-		(at 116.84 73.66 0)
-		(unit 1)
-		(body_style 1)
-		(exclude_from_sim no)
-		(in_bom yes)
-		(on_board yes)
-		(in_pos_files yes)
-		(dnp no)
-		(property "Reference" "#PWR072"
-			(at 116.84 77.47 0)
-			(hide yes)
-			(show_name no)
-			(do_not_autoplace no)
-			(effects
-				(font
-					(size 1.27 1.27)
-				)
-			)
-		)
-		(property "Value" "+5VA"
-			(at 117.221 69.2658 0)
-			(show_name no)
-			(do_not_autoplace no)
-			(effects
-				(font
-					(size 1.27 1.27)
-				)
-			)
-		)
-		(property "Footprint" ""
-			(at 116.84 73.66 0)
-			(hide yes)
-			(show_name no)
-			(do_not_autoplace no)
-			(effects
-				(font
-					(size 1.27 1.27)
-				)
-			)
-		)
-		(property "Datasheet" ""
-			(at 116.84 73.66 0)
-			(hide yes)
-			(show_name no)
-			(do_not_autoplace no)
-			(effects
-				(font
-					(size 1.27 1.27)
-				)
-			)
-		)
-		(property "Description" ""
-			(at 116.84 73.66 0)
-			(show_name no)
-			(do_not_autoplace no)
-			(effects
-				(font
-					(size 1.27 1.27)
-				)
-			)
-		)
-		(pin "1"
-		)
-		(instances
-			(project "VESC6_OPEN_HARDWARE"
-				(path "/8bc2c25a-a1f1-4ce8-b96a-a4f8f4c35079/00000000-0000-0000-0000-00005aeaa308"
-					(reference "#PWR072")
-					(unit 1)
-				)
-			)
-		)
-	)
-	(symbol
-		(lib_id "power:VCC")
-		(at 166.37 73.66 0)
-		(unit 1)
-		(body_style 1)
-		(exclude_from_sim no)
-		(in_bom yes)
-		(on_board yes)
-		(in_pos_files yes)
-		(dnp no)
-		(property "Reference" "#PWR073"
-			(at 166.37 77.47 0)
-			(hide yes)
-			(show_name no)
-			(do_not_autoplace no)
-			(effects
-				(font
-					(size 1.27 1.27)
-				)
-			)
-		)
-		(property "Value" "+3V3a"
-			(at 166.8018 69.2658 0)
-			(show_name no)
-			(do_not_autoplace no)
-			(effects
-				(font
-					(size 1.27 1.27)
-				)
-			)
-		)
-		(property "Footprint" ""
-			(at 166.37 73.66 0)
-			(hide yes)
-			(show_name no)
-			(do_not_autoplace no)
-			(effects
-				(font
-					(size 1.27 1.27)
-				)
-			)
-		)
-		(property "Datasheet" ""
-			(at 166.37 73.66 0)
-			(hide yes)
-			(show_name no)
-			(do_not_autoplace no)
-			(effects
-				(font
-					(size 1.27 1.27)
-				)
-			)
-		)
-		(property "Description" ""
-			(at 166.37 73.66 0)
-			(show_name no)
-			(do_not_autoplace no)
-			(effects
-				(font
-					(size 1.27 1.27)
-				)
-			)
-		)
-		(pin "1"
-		)
-		(instances
-			(project "VESC6_OPEN_HARDWARE"
-				(path "/8bc2c25a-a1f1-4ce8-b96a-a4f8f4c35079/00000000-0000-0000-0000-00005aeaa308"
-					(reference "#PWR073")
+				(path "/8bc2c25a-a1f1-4ce8-b96a-a4f8f4c35079/1e81ec4a-7813-42c9-8244-ecd5bd9e7dba/b2b9706e-bd8f-4858-b41c-0ad60782e278"
+					(reference "U1002")
 					(unit 1)
 				)
@@
 		(instances
 			(project "VESC6_OPEN_HARDWARE"
-				(path "/8bc2c25a-a1f1-4ce8-b96a-a4f8f4c35079/00000000-0000-0000-0000-00005aeaa308"
+				(path "/8bc2c25a-a1f1-4ce8-b96a-a4f8f4c35079/1e81ec4a-7813-42c9-8244-ecd5bd9e7dba/b2b9706e-bd8f-4858-b41c-0ad60782e278"
 					(reference "#PWR074")
 					(unit 1)

Commit message: relinked UUIDs
Parts:
- renumbered C1004 to C101, C1005 to C102, R1012 to R101, U1002 to U101
Changed lines of the file:
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@@
 		(in_pos_files yes)
 		(dnp no)
-		(property "Reference" "C1004"
+		(property "Reference" "C101"
 			(at 118.11 87.63 0)
 			(show_name no)
@@
 			(project "VESC6_OPEN_HARDWARE"
 				(path "/8bc2c25a-a1f1-4ce8-b96a-a4f8f4c35079/1e81ec4a-7813-42c9-8244-ecd5bd9e7dba/b2b9706e-bd8f-4858-b41c-0ad60782e278"
-					(reference "C1004")
+					(reference "C101")
 					(unit 1)
 				)
@@
 		(in_pos_files yes)
 		(dnp no)
-		(property "Reference" "C1005"
+		(property "Reference" "C102"
 			(at 168.91 88.9 0)
 			(show_name no)
@@
 			(project "VESC6_OPEN_HARDWARE"
 				(path "/8bc2c25a-a1f1-4ce8-b96a-a4f8f4c35079/1e81ec4a-7813-42c9-8244-ecd5bd9e7dba/b2b9706e-bd8f-4858-b41c-0ad60782e278"
-					(reference "C1005")
+					(reference "C102")
 					(unit 1)
 				)
@@
 		(in_pos_files yes)
 		(dnp no)
-		(property "Reference" "R1012"
+		(property "Reference" "R101"
 			(at 181.61 82.55 90)
 			(show_name no)
@@
 			(project "VESC6_OPEN_HARDWARE"
 				(path "/8bc2c25a-a1f1-4ce8-b96a-a4f8f4c35079/1e81ec4a-7813-42c9-8244-ecd5bd9e7dba/b2b9706e-bd8f-4858-b41c-0ad60782e278"
-					(reference "R1012")
+					(reference "R101")
 					(unit 1)
 				)
@@
 		(in_pos_files yes)
 		(dnp no)
-		(property "Reference" "U1002"
+		(property "Reference" "U101"
 			(at 145.415 70.739 0)
 			(show_name no)
@@
 			(project "VESC6_OPEN_HARDWARE"
 				(path "/8bc2c25a-a1f1-4ce8-b96a-a4f8f4c35079/1e81ec4a-7813-42c9-8244-ecd5bd9e7dba/b2b9706e-bd8f-4858-b41c-0ad60782e278"
-					(reference "U1002")
+					(reference "U101")
 					(unit 1)
 				)

Commit message: it seems to work. yay
Parts:
- renumbered C101 to C1001, C102 to C1002, R101 to R1001, U101 to U1001
Changed lines of the file:
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@@
 		(in_pos_files yes)
 		(dnp no)
-		(property "Reference" "C101"
+		(property "Reference" "C1001"
 			(at 118.11 87.63 0)
 			(show_name no)
@@
 			(project "VESC6_OPEN_HARDWARE"
 				(path "/8bc2c25a-a1f1-4ce8-b96a-a4f8f4c35079/1e81ec4a-7813-42c9-8244-ecd5bd9e7dba/b2b9706e-bd8f-4858-b41c-0ad60782e278"
-					(reference "C101")
+					(reference "C1001")
+					(unit 1)
+				)
+				(path "/8bc2c25a-a1f1-4ce8-b96a-a4f8f4c35079/cc03c9bc-7d6e-4340-8742-d977d081ffa4/3cba2e60-3b85-4d67-b7ac-7f0744ce8fec"
+					(reference "C2001")
 					(unit 1)
 				)
@@
 		(in_pos_files yes)
 		(dnp no)
-		(property "Reference" "C102"
+		(property "Reference" "C1002"
 			(at 168.91 88.9 0)
 			(show_name no)
@@
 			(project "VESC6_OPEN_HARDWARE"
 				(path "/8bc2c25a-a1f1-4ce8-b96a-a4f8f4c35079/1e81ec4a-7813-42c9-8244-ecd5bd9e7dba/b2b9706e-bd8f-4858-b41c-0ad60782e278"
-					(reference "C102")
+					(reference "C1002")
+					(unit 1)
+				)
+				(path "/8bc2c25a-a1f1-4ce8-b96a-a4f8f4c35079/cc03c9bc-7d6e-4340-8742-d977d081ffa4/3cba2e60-3b85-4d67-b7ac-7f0744ce8fec"
+					(reference "C2002")
 					(unit 1)
 				)
@@
 		(in_pos_files yes)
 		(dnp no)
-		(property "Reference" "R101"
+		(property "Reference" "R1001"
 			(at 181.61 82.55 90)
 			(show_name no)
@@
 			(project "VESC6_OPEN_HARDWARE"
 				(path "/8bc2c25a-a1f1-4ce8-b96a-a4f8f4c35079/1e81ec4a-7813-42c9-8244-ecd5bd9e7dba/b2b9706e-bd8f-4858-b41c-0ad60782e278"
-					(reference "R101")
+					(reference "R1001")
+					(unit 1)
+				)
+				(path "/8bc2c25a-a1f1-4ce8-b96a-a4f8f4c35079/cc03c9bc-7d6e-4340-8742-d977d081ffa4/3cba2e60-3b85-4d67-b7ac-7f0744ce8fec"
+					(reference "R2001")
 					(unit 1)
 				)
@@
 		(in_pos_files yes)
 		(dnp no)
-		(property "Reference" "U101"
+		(property "Reference" "U1001"
 			(at 145.415 70.739 0)
 			(show_name no)
@@
 			(project "VESC6_OPEN_HARDWARE"
 				(path "/8bc2c25a-a1f1-4ce8-b96a-a4f8f4c35079/1e81ec4a-7813-42c9-8244-ecd5bd9e7dba/b2b9706e-bd8f-4858-b41c-0ad60782e278"
-					(reference "U101")
+					(reference "U1001")
+					(unit 1)
+				)
+				(path "/8bc2c25a-a1f1-4ce8-b96a-a4f8f4c35079/cc03c9bc-7d6e-4340-8742-d977d081ffa4/3cba2e60-3b85-4d67-b7ac-7f0744ce8fec"
+					(reference "U2001")
 					(unit 1)
 				)
@@
 		(in_pos_files yes)
 		(dnp no)
-		(property "Reference" "#PWR074"
+		(property "Reference" "#PWR01001"
 			(at 166.37 111.76 0)
 			(hide yes)
@@
 			(project "VESC6_OPEN_HARDWARE"
 				(path "/8bc2c25a-a1f1-4ce8-b96a-a4f8f4c35079/1e81ec4a-7813-42c9-8244-ecd5bd9e7dba/b2b9706e-bd8f-4858-b41c-0ad60782e278"
-					(reference "#PWR074")
-					(unit 1)
-				)
+					(reference "#PWR01001")
+					(unit 1)
+				)
+				(path "/8bc2c25a-a1f1-4ce8-b96a-a4f8f4c35079/cc03c9bc-7d6e-4340-8742-d977d081ffa4/3cba2e60-3b85-4d67-b7ac-7f0744ce8fec"
+					(reference "#PWR02001")
+					(unit 1)
+				)

Commit message: finishing touches
Parts:
- C1001, C1002: LCSC (none) -> C23630; LCSC part no. C23630 -> (none)
- R1001: LCSC (none) -> C22787; LCSC part no. C22787 -> (none)
- U1001: LCSC (none) -> C124020; LCSC part no. C124020 -> (none)
Changed lines of the file:
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@@
-			)
-		)
-		(property "LCSC part no." "C23630"
-			(at 116.84 90.17 0)
-			(hide yes)
-			(show_name no)
-			(do_not_autoplace no)
-			(effects
-				(font
-					(size 1.27 1.27)
-				)
 			)
 		)
@@
 		)
 		(property "MFP" "CL10A225KO8NNNC"
+			(at 116.84 90.17 0)
+			(hide yes)
+			(show_name no)
+			(do_not_autoplace no)
+			(effects
+				(font
+					(size 1.27 1.27)
+				)
+			)
+		)
+		(property "LCSC" "C23630"
 			(at 116.84 90.17 0)
 			(hide yes)
@@
 			)
 		)
-		(property "LCSC part no." "C23630"
-			(at 166.37 91.44 0)
-			(hide yes)
-			(show_name no)
-			(do_not_autoplace no)
-			(effects
-				(font
-					(size 1.27 1.27)
-				)
-			)
-		)
 		(property "Critical" "N"
 			(at 166.37 91.44 0)
@@
 		)
 		(property "MFP" "CL10A225KO8NNNC"
+			(at 166.37 91.44 0)
+			(hide yes)
+			(show_name no)
+			(do_not_autoplace no)
+			(effects
+				(font
+					(size 1.27 1.27)
+				)
+			)
+		)
+		(property "LCSC" "C23630"
 			(at 166.37 91.44 0)
 			(hide yes)
@@
 			)
 		)
-		(property "LCSC part no." "C22787"
-			(at 179.07 81.28 0)
-			(hide yes)
-			(show_name no)
-			(do_not_autoplace no)
-			(effects
-				(font
-					(size 1.27 1.27)
-				)
-			)
-		)
 		(property "Critical" "N"
 			(at 179.07 81.28 0)
@@
 		(property "MFP" "0603WAF1200T5E"
 			(at 179.07 81.28 0)
+			(hide yes)
+			(show_name no)
+			(do_not_autoplace no)
+			(effects
+				(font
+					(size 1.27 1.27)
+				)
+			)
+		)
+		(property "LCSC" "C22787"
+			(at 179.07 81.28 90)
 			(hide yes)
 			(show_name no)
@@
 			)
 		)
-		(property "LCSC part no." "C124020"
-			(at 147.32 82.55 0)
-			(hide yes)
-			(show_name no)
-			(do_not_autoplace no)
-			(effects
-				(font
-					(size 1.27 1.27)
-				)
-			)
-		)
 		(property "Critical" "Y"
 			(at 147.32 82.55 0)
@@
 			(at 147.32 82.55 0)
 			(hide yes)
+			(show_name no)
+			(do_not_autoplace no)
+			(effects
+				(font
+					(size 1.27 1.27)
+				)
+			)
+		)
+		(property "LCSC" "C124020"
+			(at 147.32 82.55 0)
+			(hide yes)

Commit message: more tweaks
Other:
- company: (none) -> craigg96, Tomáš Kuchta
- title: (none) -> 2ch VESC based on VESC6
Changed lines of the file:
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@@
 	(paper "A4")
 	(title_block
+		(title "2ch VESC based on VESC6")
 		(date "2025-03-23")
-		(rev "A")
-		(comment 1 "Drawn By: CG")
+		(rev "B")
+		(company "craigg96, Tomáš Kuchta")
 	)
 	(junction
