File: CHa.kicad_sch (KiCad schematic)
At the start: 17 parts, among them P1001 CAN 2, P1002 SWD, P1003 CAN 1, P1004 HALL/Encoder, P1005 ADC_SWITCH

Commit message: relinked UUIDs
Parts:
- renumbered C1001 to C148, D1001 to D103, D1002 to D104, P1001 to P104, P1003 to P105, P1002 to P106, P1004 to P107, P1005 to P108, R1001 to R134, R1002 to R135, R1003 to R136, R1004 to R137, R1005 to R138, R1006 to R139, R1007 to R140, R1008 to R141, R1009 to R142

Commit message: it seems to work. yay
Parts:
- renumbered C148 to C301, D103 to D301, D104 to D302, P104 to P301, P105 to P302, P106 to P303, P107 to P304, P108 to P305, R134 to R301, R135 to R302, R136 to R303, R137 to R304, R138 to R305, R139 to R306, R140 to R307, R141 to R308, R142 to R309

Commit message: small improvements.
Parts:
- P301, P302, P305: LCSC part no. C23390337 -> C160404
Connections:
- net CAN/CANH renamed CANH
- net CAN/CANL renamed CANL
Changed lines of the file:
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@@
 	)
 	(junction
+		(at 35.56 58.42)
+		(diameter 0)
+		(color 0 0 0 0)
+	)
+	(junction
+		(at 35.56 60.96)
+		(diameter 0)
+		(color 0 0 0 0)
+	)
+	(junction
 		(at 81.28 109.22)
 		(diameter 0)
@@
 	(wire
 		(pts
+			(xy 26.67 60.96) (xy 35.56 60.96)
+		)
+		(stroke
+			(width 0)
+			(type default)
+		)
+	)
+	(wire
+		(pts
 			(xy 162.56 48.26) (xy 177.8 48.26)
 		)
@@
 	(wire
 		(pts
+			(xy 26.67 58.42) (xy 35.56 58.42)
+		)
+		(stroke
+			(width 0)
+			(type default)
+		)
+	)
+	(wire
+		(pts
 			(xy 100.33 137.16) (xy 106.68 137.16)
 		)
@@
 		)
 	)
+	(label "CANL"
+		(at 54.61 58.42 0)
+		(effects
+			(font
+				(size 1.27 1.27)
+			)
+			(justify left bottom)
+		)
+	)
+	(label "CANH"
+		(at 54.61 60.96 0)
+		(effects
+			(font
+				(size 1.27 1.27)
+			)
+			(justify left bottom)
+		)
+	)
+	(hierarchical_label "CANL"
+		(shape bidirectional)
+		(at 26.67 58.42 180)
+		(effects
+			(font
+				(size 1.27 1.27)
+			)
+			(justify right)
+		)
+	)
+	(hierarchical_label "CANH"
+		(shape bidirectional)
+		(at 26.67 60.96 180)
+		(effects
+			(font
+				(size 1.27 1.27)
+			)
+			(justify right)
+		)
+	)
 	(symbol
 		(lib_id "power:+5V")
@@
 		)
 		(property "Value" "CAN 1"
-			(at 48.26 68.58 0)
+			(at 47.752 67.818 0)
 			(show_name no)
 			(do_not_autoplace no)
@@
 			)
 		)
-		(property "LCSC part no." "C23390337"
+		(property "LCSC part no." "C160404"
 			(at 49.53 60.96 0)
 			(hide yes)
@@
 		)
 		(property "Value" "CAN 2"
-			(at 29.21 68.58 0)
+			(at 28.702 68.072 0)
 			(show_name no)
 			(do_not_autoplace no)
@@
 			)
 		)
-		(property "LCSC part no." "C23390337"
+		(property "LCSC part no." "C160404"
 			(at 30.48 60.96 0)
 			(hide yes)
@@
 			)
 		)
-		(property "LCSC part no." "C23390337"
+		(property "LCSC part no." "C160404"
 			(at 119.38 21.59 0)
 			(hide yes)

Commit message: finishing touches
Parts:
- C301: LCSC (none) -> C14663; LCSC part no. C14663 -> (none)
- D301: LCSC (none) -> C2286; LCSC part no. C2286 -> (none)
- D302: LCSC (none) -> C2290; LCSC part no. C2290 -> (none)
- P301, P302, P305: LCSC (none) -> C160404; LCSC part no. C160404 -> (none)
- P303, P304: LCSC (none) -> C160405; LCSC part no. C160405 -> (none)
- R301, R302, R303: LCSC (none) -> C4190; LCSC part no. C4190 -> (none)
- R305, R306: LCSC (none) -> C23345; LCSC part no. C23345 -> (none)
- R307: LCSC (none) -> C25804; LCSC part no. C25804 -> (none)
- R308, R309: LCSC (none) -> C22787; LCSC part no. C22787 -> (none)

Commit message: more tweaks
Other:
- company: (none) -> craigg96, Tomáš Kuchta
- title: (none) -> 2ch VESC based on VESC6
Changed lines of the file:
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@@
 	(paper "A4")
 	(title_block
-		(rev "A")
+		(title "2ch VESC based on VESC6")
+		(rev "B")
+		(company "craigg96, Tomáš Kuchta")
 	)
 	(junction
