File: CHb.kicad_sch (KiCad schematic)
At the start: 0 parts

Commit message: it seems to work. yay
Parts:
- added C401: 100n, Capacitor_SMD:C_0603_1608Metric, symbol Device:C
- added D401: RED, Diode_SMD:D_0603_1608Metric, symbol Device:LED
- added D402: WHITE, Diode_SMD:D_0603_1608Metric, symbol Device:LED
- added P401: CAN 2, Connector_JST:JST_SH_SM04B-SRSS-TB_1x04-1MP_P1.00mm_Horizontal, symbol Connector_Generic_MountingPin:Conn_01x04_MountingPin
- added P402: CAN 1, Connector_JST:JST_SH_SM04B-SRSS-TB_1x04-1MP_P1.00mm_Horizontal, symbol Connector_Generic_MountingPin:Conn_01x04_MountingPin
- added P403: SWD, Connector_JST:JST_SH_SM06B-SRSS-TB_1x06-1MP_P1.00mm_Horizontal, symbol Connector_Generic_MountingPin:Conn_01x06_MountingPin
- added P404: HALL/Encoder, Connector_JST:JST_SH_SM06B-SRSS-TB_1x06-1MP_P1.00mm_Horizontal, symbol Connector_Generic_MountingPin:Conn_01x06_MountingPin
- added P405: ADC_SWITCH, Connector_JST:JST_SH_SM04B-SRSS-TB_1x04-1MP_P1.00mm_Horizontal, symbol Connector_Generic_MountingPin:Conn_01x04_MountingPin
- added R401, R402, R403: 2k2, Resistor_SMD:R_0603_1608Metric, symbol Device:R
- added R404: DNP, Resistor_SMD:R_0603_1608Metric, symbol Device:R
- added R405, R406: 22R, Resistor_SMD:R_0603_1608Metric, symbol Device:R
- added R407: 10k, Resistor_SMD:R_0603_1608Metric, symbol Device:R
- added R408, R409: 120R, Resistor_SMD:R_0603_1608Metric, symbol Device:R
Connections:
- new net: D402.1 (K), R409.1
- new net: D401.1 (K), R408.1
- new net +3V3a: P403.6 (Pin_6), R407.1
- new net +5Va: P401.4 (Pin_4), P402.4 (Pin_4), P403.1 (Pin_1), P404.6 (Pin_6), P405.4 (Pin_4), R401.2, R402.2, R403.2, R404.1
- new net CAN/CANH: P401.2 (Pin_2), P402.2 (Pin_2)
- new net CAN/CANL: P401.1 (Pin_1), P402.1 (Pin_1)
- new net DRV8301/SWITCH-: P405.1 (Pin_1)
- new net GND: C401.1, P401.3 (Pin_3), P401.MP (MountPin), P402.3 (Pin_3), P402.MP (MountPin), P403.4 (Pin_4), P403.MP (MountPin), P404.1 (Pin_1), P404.MP (MountPin), P405.3 (Pin_3), P405.MP (MountPin), R408.2, R409.2
- new net USB/USB_D+: R406.2
- new net USB/USB_D-: R405.2
- new net USB/VBUS: R404.2
- new net stm32f40x/HALL_1: P404.4 (Pin_4), R401.1
- new net stm32f40x/HALL_2: P404.3 (Pin_3), R402.1
- new net stm32f40x/HALL_3: P404.2 (Pin_2), R403.1
- new net stm32f40x/LED_GREEN: D402.2 (A)
- new net stm32f40x/LED_RED: D401.2 (A)
- new net stm32f40x/NRST: P403.2 (Pin_2)
- new net stm32f40x/SCK_ADC_EXT: P405.2 (Pin_2)
- new net stm32f40x/SWCLK: P403.5 (Pin_5)
- new net stm32f40x/SWDIO: P403.3 (Pin_3)
- new net stm32f40x/TEMP_MOTOR: C401.2, P404.5 (Pin_5), R407.2
- new net stm32f40x/USB_DM: R405.1
- new net stm32f40x/USB_DP: R406.1
Other:
- added sheet CAN (CAN.kicad_sch)
- added sheet DRV8301 (DRV8301.kicad_sch)
- added sheet Hbridge (Hbridge.kicad_sch)
- added sheet IMU (IMU.kicad_sch)
- added sheet USB (USB.kicad_sch)
- added sheet stm32f40x (mcu.kicad_sch)

Commit message: it looks like it's going together well!!!
Connections:
- net +3V3a renamed +3V3b
- net +5Va renamed +5Vb
Changed lines of the file:
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@@
 			)
 		)
-		(property "Value" "+3V3a"
+		(property "Value" "+3V3b"
 			(at 99.06 97.79 0)
 			(show_name no)
@@
 			)
 		)
-		(property "Value" "+5Va"
+		(property "Value" "+5Vb"
 			(at 62.9412 66.421 90)
 			(show_name no)
@@
 			)
 		)
-		(property "Value" "+3V3a"
+		(property "Value" "+3V3b"
 			(at 149.0218 28.6258 0)
 			(show_name no)
@@
 			)
 		)
-		(property "Value" "+5Va"
+		(property "Value" "+5Vb"
 			(at 89.281 48.9458 0)
 			(show_name no)
@@
 			)
 		)
-		(property "Value" "+3V3a"
+		(property "Value" "+3V3b"
 			(at 196.0118 28.6258 0)
 			(show_name no)
@@
 			)
 		)
-		(property "Value" "+5Va"
+		(property "Value" "+5Vb"
 			(at 130.1242 27.051 90)
 			(show_name no)
@@
 			)
 		)
-		(property "Value" "+5Va"
+		(property "Value" "+5Vb"
 			(at 65.4812 160.401 90)
 			(show_name no)
@@
 			)
 		)
-		(property "Value" "+3V3a"
+		(property "Value" "+3V3b"
 			(at 81.7118 48.9458 0)
 			(show_name no)
@@
 			)
 		)
-		(property "Value" "+5Va"
+		(property "Value" "+5Vb"
 			(at 202.311 28.6258 0)
 			(show_name no)
@@
 			)
 		)
-		(property "Value" "+3V3a"
+		(property "Value" "+3V3b"
 			(at 87.63 127 0)
 			(show_name no)
@@
 			)
 		)
-		(property "Value" "+5Va"
+		(property "Value" "+5Vb"
 			(at 37.211 89.5858 0)
 			(show_name no)
@@
 			)
 		)
-		(property "Value" "+3V3a"
+		(property "Value" "+3V3b"
 			(at 241.7318 28.6258 0)
 			(show_name no)
@@
 			)
 		)
-		(property "Value" "+3V3a"
+		(property "Value" "+3V3b"
 			(at 73.1012 147.7518 90)
 			(show_name no)
@@
 			)
 		)
-		(property "Value" "+5Va"
+		(property "Value" "+5Vb"
 			(at 94.361 23.5458 0)
 			(show_name no)

Commit message: small improvements.
Parts:
- removed P401: CAN 2, Connector_JST:JST_SH_SM04B-SRSS-TB_1x04-1MP_P1.00mm_Horizontal, symbol Connector_Generic_MountingPin:Conn_01x04_MountingPin
- P401: renamed from P402; footprint Connector_JST:JST_SH_SM04B-SRSS-TB_1x04-1MP_P1.00mm_Horizontal -> Connector_JST:JST_SH_BM04B-SRSS-TB_1x04-1MP_P1.00mm_Vertical; LCSC part no. C23390337 -> C160390
- P403: footprint Connector_JST:JST_SH_SM06B-SRSS-TB_1x06-1MP_P1.00mm_Horizontal -> Connector_JST:JST_SH_BM06B-SRSS-TB_1x06-1MP_P1.00mm_Vertical; LCSC part no. C160405 -> C160392
- P405: footprint Connector_JST:JST_SH_SM04B-SRSS-TB_1x04-1MP_P1.00mm_Horizontal -> Connector_JST:JST_SH_BM04B-SRSS-TB_1x04-1MP_P1.00mm_Vertical; LCSC part no. C23390337 -> C160390
Connections:
- net CAN/CANH renamed CANH
- net CAN/CANL renamed CANL

Commit message: finishing touches
Parts:
- C401: LCSC (none) -> C14663; LCSC part no. C14663 -> (none)
- D401: LCSC (none) -> C2286; LCSC part no. C2286 -> (none)
- D402: LCSC (none) -> C2290; LCSC part no. C2290 -> (none)
- P401, P405: LCSC (none) -> C160390; LCSC part no. C160390 -> (none)
- P403: LCSC (none) -> C160392; LCSC part no. C160392 -> (none)
- P404: LCSC (none) -> C160405; LCSC part no. C160405 -> (none)
- R401, R402, R403: LCSC (none) -> C4190; LCSC part no. C4190 -> (none)
- R405, R406: LCSC (none) -> C23345; LCSC part no. C23345 -> (none)
- R407: LCSC (none) -> C25804; LCSC part no. C25804 -> (none)
- R408, R409: LCSC (none) -> C22787; LCSC part no. C22787 -> (none)

Commit message: more tweaks
Other:
- company: (none) -> craigg96, Tomáš Kuchta
- title: (none) -> 2ch VESC based on VESC6
Changed lines of the file:
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@@
 	(paper "A4")
 	(title_block
-		(rev "A")
+		(title "2ch VESC based on VESC6")
+		(rev "B")
+		(company "craigg96, Tomáš Kuchta")
 	)
 	(junction
