File: DRV8301.kicad_sch (KiCad schematic)
At the start: 39 parts, among them U2 LM3671, U3 DRV8301

Commit message: prep for chaneling. fixed the connector references, added cha to this schematic.
Connections:
- net +5V renamed +5VA
- net VCC renamed +3V3a
Changed lines of the file:
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@@
 			)
 		)
-		(property "Value" "+5V"
+		(property "Value" "+5VA"
 			(at 81.661 34.9758 0)
 			(show_name no)
@@
 			)
 		)
-		(property "Value" "+5V"
+		(property "Value" "+5VA"
 			(at 209.931 43.8658 0)
 			(show_name no)
@@
 			)
 		)
-		(property "Value" "VCC"
+		(property "Value" "+3V3a"
 			(at 169.3418 51.4858 0)
 			(show_name no)
@@
 			)
 		)
-		(property "Value" "+5V"
+		(property "Value" "+5VA"
 			(at 248.031 26.0858 0)
 			(show_name no)
@@
 			)
 		)
-		(property "Value" "VCC"
+		(property "Value" "+3V3a"
 			(at 129.9718 136.5758 0)
 			(show_name no)
@@
 			)
 		)
-		(property "Value" "+5V"
+		(property "Value" "+5VA"
 			(at 84.201 137.8458 0)
 			(show_name no)

Commit message: more fixes for channels
Parts:
- renumbered C13 to C1017, C14 to C1018, C15 to C1019, C17 to C1020, C16 to C1021, C20 to C1022, C18 to C1023, C19 to C1024, C64 to C1025, C21 to C1026, C22 to C1027, C26 to C1028, C23 to C1029, C24 to C1030, C25 to C1031, C28 to C1032, C27 to C1033, C31 to C1034, C32 to C1035, D4 to D1003, D5 to D1004, L1 to L1001, L2 to L1002, R10 to R1013, R11 to R1014, R12 to R1015, R13 to R1016, R14 to R1017, R38 to R1018, R15 to R1019, R16 to R1020, R17 to R1021, R18 to R1022, R19 to R1023, R20 to R1024, R21 to R1025, R22 to R1026, U2 to U1004, U3 to U1005
Connections:
- net +3V3a renamed +3V3
- net +5VA renamed +5V
Other:
- moved on the sheet: C1017, C1026, C1035

Commit message: relinked UUIDs
Parts:
- renumbered C1017 to C103, C1018 to C104, C1019 to C105, C1020 to C106, C1021 to C107, C1022 to C108, C1023 to C109, C1024 to C110, C1025 to C111, C1026 to C112, C1027 to C113, C1028 to C114, C1029 to C115, C1030 to C116, C1031 to C117, C1032 to C118, C1033 to C119, C1034 to C120, C1035 to C121, D1003 to D101, D1004 to D102, L1001 to L101, L1002 to L102, R1013 to R102, R1014 to R103, R1015 to R104, R1016 to R105, R1017 to R106, R1018 to R107, R1019 to R108, R1020 to R109, R1021 to R110, R1022 to R111, R1023 to R112, R1024 to R113, R1025 to R114, R1026 to R115, U1004 to U102, U1005 to U103

Commit message: it seems to work. yay
Parts:
- renumbered C103 to C1101, C104 to C1102, C105 to C1103, C106 to C1104, C107 to C1105, C108 to C1106, C109 to C1107, C110 to C1108, C111 to C1109, C112 to C1110, C113 to C1111, C114 to C1112, C115 to C1113, C116 to C1114, C117 to C1115, C118 to C1116, C119 to C1117, C120 to C1118, C121 to C1119, D101 to D1101, D102 to D1102, L101 to L1101, L102 to L1102, R102 to R1101, R103 to R1102, R104 to R1103, R105 to R1104, R106 to R1105, R107 to R1106, R108 to R1107, R109 to R1108, R110 to R1109, R111 to R1110, R112 to R1111, R113 to R1112, R114 to R1113, R115 to R1114, U102 to U1101, U103 to U1102

Commit message: finishing touches
Parts:
- C1101, C1102, C1103, C1104, C1106, C1109, C1118: LCSC (none) -> C23630; LCSC part no. C23630 -> (none)
- C1105: LCSC (none) -> C1631; LCSC part no. C1631 -> (none)
- C1107: LCSC (none) -> C107035; LCSC part no. C107035 -> (none)
- C1108: LCSC (none) -> C21122; LCSC part no. C21122 -> (none)
- C1110, C1119: LCSC (none) -> C16133; LCSC part no. C16133 -> (none)
- C1111: LCSC (none) -> C1596; LCSC part no. C1596 -> (none)
- C1112, C1117: LCSC (none) -> C385987; LCSC part no. C385987 -> (none)
- C1113, C1114, C1115: LCSC (none) -> C21120; LCSC part no. C21120 -> (none)
- C1116: LCSC (none) -> C14663; LCSC part no. C14663 -> (none)
- D1101: LCSC (none) -> C2923951; LCSC part no. C2923951 -> (none)
- D1102: LCSC (none) -> C129544; LCSC part no. C129544 -> (none)
- L1101: LCSC (none) -> C383398; LCSC part no. C383398 -> (none)
- L1102: LCSC (none) -> C266430; LCSC part no. C266430 -> (none)
- R1101: LCSC (none) -> C22978; LCSC part no. C22978 -> (none)
- R1102: LCSC (none) -> C25810; LCSC part no. C25810 -> (none)
- R1103: LCSC (none) -> C22809; LCSC part no. C22809 -> (none)
- R1104, R1106: LCSC (none) -> C25804; LCSC part no. C25804 -> (none)
- R1105: LCSC (none) -> C22961; LCSC part no. C22961 -> (none)
- R1107, R1109, R1111, R1113: LCSC (none) -> C23153; LCSC part no. C23153 -> (none)
- R1108, R1110, R1112, R1114: LCSC (none) -> C4190; LCSC part no. C4190 -> (none)
- U1101: LCSC (none) -> C477918; LCSC part no. C477918 -> (none)
- U1102: LCSC (none) -> C98969; LCSC part no. C98969 -> (none)

Commit message: more tweaks
Other:
- company: (none) -> craigg96, Tomáš Kuchta
- title: (none) -> 2ch VESC based on VESC6
Changed lines of the file:
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@@
 	(paper "A4")
 	(title_block
+		(title "2ch VESC based on VESC6")
 		(date "2025-03-23")
-		(rev "A")
-		(comment 1 "Drawn By: CG")
+		(rev "B")
+		(company "craigg96, Tomáš Kuchta")
 	)
 	(junction
