File: Hbridge.kicad_sch (KiCad schematic)
At the start: 45 parts, among them P10 PH_A, P11 SUPPLY, P12 GND, P8 PH_C, P9 PH_B, Q1 STL130N6F7, Q2 STL130N6F7, Q3 STL130N6F7, Q4 STL130N6F7, Q5 STL130N6F7, Q6 STL130N6F7, U5 AD8418, U6 AD8418, U7 AD8418

Commit message: more fixes for channels
Parts:
- removed C48, C49, C50, C51: 220u_63v, Capacitor_SMD:CP_Elec_10x10.5, symbol Device:C
- removed P11: SUPPLY, Connector_Pin:Pin_D1.0mm_L10.0mm_LooseFit, symbol Connector_Generic:Conn_01x01
- removed P12: GND, Connector_Pin:Pin_D1.0mm_L10.0mm_LooseFit, symbol Connector_Generic:Conn_01x01
- C1040: renamed from C37; LCSC part no. C385986 -> C385987; Link https://jlcpcb.com/partdetail/TaiyoYuden-HMK325C7475KMHPE/C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 -> (none); MFP HMK325C7475KMHPE -> (none)
- C1041: renamed from C39; LCSC part no. C385986 -> C385987; Link https://jlcpcb.com/partdetail/TaiyoYuden-HMK325C7475KMHPE/C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 -> (none); MFP HMK325C7475KMHPE -> (none)
- C1044: renamed from C40; LCSC part no. C385986 -> C385987; Link https://jlcpcb.com/partdetail/TaiyoYuden-HMK325C7475KMHPE/C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 -> (none); MFP HMK325C7475KMHPE -> (none)
- C1045: renamed from C41; LCSC part no. C385986 -> C385987; Link https://jlcpcb.com/partdetail/TaiyoYuden-HMK325C7475KMHPE/C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 -> (none); MFP HMK325C7475KMHPE -> (none)
- C1051: renamed from C43; LCSC part no. C385986 -> C385987; Link https://jlcpcb.com/partdetail/TaiyoYuden-HMK325C7475KMHPE/C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 -> (none); MFP HMK325C7475KMHPE -> (none)
- C1052: renamed from C44; LCSC part no. C385986 -> C385987; Link https://jlcpcb.com/partdetail/TaiyoYuden-HMK325C7475KMHPE/C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 -> (none); MFP HMK325C7475KMHPE -> (none)
- P1006: renamed from P8; LCSC part no. (none) -> C7200700
- P1007: renamed from P9; LCSC part no. (none) -> C7200700
- P1008: renamed from P10; LCSC part no. (none) -> C7200700
- renumbered C35 to C1036, C29 to C1037, C30 to C1038, C45 to C1039, C38 to C1042, C36 to C1043, C42 to C1046, Q1 to Q1001, Q2 to Q1002, Q3 to Q1003, Q4 to Q1004, Q5 to Q1005, Q6 to Q1006, R24 to R1029, R25 to R1030, R26 to R1031, R35 to R1032, R36 to R1033, R37 to R1034, R29 to R1035, R27 to R1036, R28 to R1037, R30 to R1038, R31 to R1039, R32 to R1040, R33 to R1041, R34 to R1042, U5 to U1007, U6 to U1008, U7 to U1009
Connections:
- net VCC renamed +3V3

Commit message: relinked UUIDs
Parts:
- renumbered C1036 to C122, C1037 to C123, C1038 to C124, C1039 to C125, C1040 to C126, C1041 to C127, C1042 to C128, C1043 to C129, C1044 to C130, C1045 to C131, C1046 to C132, C1051 to C133, C1052 to C134, P1006 to P101, P1007 to P102, P1008 to P103, Q1001 to Q101, Q1002 to Q102, Q1003 to Q103, Q1004 to Q104, Q1005 to Q105, Q1006 to Q106, R1029 to R116, R1030 to R117, R1031 to R118, R1032 to R119, R1033 to R120, R1034 to R121, R1035 to R122, R1036 to R123, R1037 to R124, R1038 to R125, R1039 to R126, R1040 to R127, R1041 to R128, R1042 to R129, U1007 to U104, U1008 to U105, U1009 to U106

Commit message: it seems to work. yay
Parts:
- renumbered C122 to C1201, C123 to C1202, C124 to C1203, C125 to C1204, C126 to C1205, C127 to C1206, C128 to C1207, C129 to C1208, C130 to C1209, C131 to C1210, C132 to C1211, C133 to C1212, C134 to C1213, P101 to P1201, P102 to P1202, P103 to P1203, Q101 to Q1201, Q102 to Q1202, Q103 to Q1203, Q104 to Q1204, Q105 to Q1205, Q106 to Q1206, R116 to R1201, R117 to R1202, R118 to R1203, R119 to R1204, R120 to R1205, R121 to R1206, R122 to R1207, R123 to R1208, R124 to R1209, R125 to R1210, R126 to R1211, R127 to R1212, R128 to R1213, R129 to R1214, U104 to U1201, U105 to U1202, U106 to U1203

Commit message: finishing touches
Parts:
- C1201, C1207, C1208, C1211: LCSC (none) -> C23630; LCSC part no. C23630 -> (none)
- C1202, C1203, C1204: LCSC (none) -> C53987; LCSC part no. C53987 -> (none)
- C1205, C1206, C1209, C1210, C1212, C1213: LCSC (none) -> C385987; LCSC part no. C385987 -> (none)
- P1201, P1202, P1203: LCSC (none) -> C7200700; LCSC part no. C7200700 -> (none)
- Q1201, Q1202, Q1203, Q1204, Q1205, Q1206: LCSC (none) -> C501008; LCSC part no. C501008 -> (none)
- R1201, R1207, R1212: LCSC (none) -> C469426; LCSC part no. C469426 -> (none)
- R1202, R1203, R1210, R1211, R1213, R1214: LCSC (none) -> C23164; LCSC part no. C23164 -> (none)
- R1204, R1205, R1206: LCSC (none) -> C22775; LCSC part no. C22775 -> (none)
- R1208: LCSC (none) -> C76589; LCSC part no. C76589 -> (none)
- R1209: LCSC (none) -> C25804; LCSC part no. C25804 -> (none)
- U1201, U1202, U1203: LCSC (none) -> C495342; LCSC part no. C495342 -> (none)

Commit message: more tweaks
Other:
- company: (none) -> craigg96, Tomáš Kuchta
- title: (none) -> 2ch VESC based on VESC6
Changed lines of the file:
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@@
 	(paper "A4")
 	(title_block
+		(title "2ch VESC based on VESC6")
 		(date "2025-03-23")
-		(rev "A")
-		(comment 1 "Drawn By: CG")
+		(rev "B")
+		(company "craigg96, Tomáš Kuchta")
 	)
 	(junction
