File: IMU.kicad_sch (KiCad schematic)
At the start: 5 parts, among them U10 LSM6DS3TR-C

Commit message: prep for chaneling. fixed the connector references, added cha to this schematic.
Connections:
- net VCC renamed +3V3a
Changed lines of the file:
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@@
 			)
 		)
-		(property "Value" "VCC"
+		(property "Value" "+3V3a"
 			(at 165.1 80.01 0)
 			(show_name no)
@@
 			)
 		)
-		(property "Value" "VCC"
+		(property "Value" "+3V3a"
 			(at 124.46 73.66 0)
 			(show_name no)

Commit message: more fixes for channels
Parts:
- renumbered C61 to C1002, C62 to C1003, R40 to R1010, R41 to R1011, U10 to U1001
Connections:
- net +3V3a renamed +3V3
Other:
- moved on the sheet: C1002, C1003

Commit message: relinked UUIDs
Parts:
- renumbered C1002 to C135, C1003 to C136, R1010 to R130, R1011 to R131, U1001 to U107
Changed lines of the file:
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@@
 		(in_pos_files yes)
 		(dnp no)
-		(property "Reference" "R1011"
+		(property "Reference" "R131"
 			(at 121.92 87.63 90)
 			(show_name no)
@@
 			(project "VESC6_OPEN_HARDWARE"
 				(path "/8bc2c25a-a1f1-4ce8-b96a-a4f8f4c35079/1e81ec4a-7813-42c9-8244-ecd5bd9e7dba/fbf84a60-b5da-4635-a9d4-00654e4ba37c"
-					(reference "R1011")
+					(reference "R131")
 					(unit 1)
 				)
@@
 		(in_pos_files yes)
 		(dnp no)
-		(property "Reference" "C1002"
+		(property "Reference" "C135"
 			(at 177.8 82.55 90)
 			(show_name no)
@@
 			(project "VESC6_OPEN_HARDWARE"
 				(path "/8bc2c25a-a1f1-4ce8-b96a-a4f8f4c35079/1e81ec4a-7813-42c9-8244-ecd5bd9e7dba/fbf84a60-b5da-4635-a9d4-00654e4ba37c"
-					(reference "C1002")
+					(reference "C135")
 					(unit 1)
 				)
@@
 		(in_pos_files yes)
 		(dnp no)
-		(property "Reference" "C1003"
+		(property "Reference" "C136"
 			(at 177.8 92.71 90)
 			(show_name no)
@@
 			(project "VESC6_OPEN_HARDWARE"
 				(path "/8bc2c25a-a1f1-4ce8-b96a-a4f8f4c35079/1e81ec4a-7813-42c9-8244-ecd5bd9e7dba/fbf84a60-b5da-4635-a9d4-00654e4ba37c"
-					(reference "C1003")
+					(reference "C136")
 					(unit 1)
 				)
@@
 		(in_pos_files yes)
 		(dnp no)
-		(property "Reference" "R1010"
+		(property "Reference" "R130"
 			(at 113.03 87.63 90)
 			(show_name no)
@@
 			(project "VESC6_OPEN_HARDWARE"
 				(path "/8bc2c25a-a1f1-4ce8-b96a-a4f8f4c35079/1e81ec4a-7813-42c9-8244-ecd5bd9e7dba/fbf84a60-b5da-4635-a9d4-00654e4ba37c"
-					(reference "R1010")
+					(reference "R130")
 					(unit 1)
 				)
@@
 		(in_pos_files yes)
 		(dnp no)
-		(property "Reference" "U1001"
+		(property "Reference" "U107"
 			(at 148.59 79.5782 0)
 			(show_name no)
@@
 			(project "VESC6_OPEN_HARDWARE"
 				(path "/8bc2c25a-a1f1-4ce8-b96a-a4f8f4c35079/1e81ec4a-7813-42c9-8244-ecd5bd9e7dba/fbf84a60-b5da-4635-a9d4-00654e4ba37c"
-					(reference "U1001")
+					(reference "U107")
 					(unit 1)
 				)

Commit message: it seems to work. yay
Parts:
- renumbered C135 to C1301, C136 to C1302, R130 to R1301, R131 to R1302, U107 to U1301
Changed lines of the file:
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@@
 		(in_pos_files yes)
 		(dnp no)
-		(property "Reference" "R131"
+		(property "Reference" "R1302"
 			(at 121.92 87.63 90)
 			(show_name no)
@@
 			(project "VESC6_OPEN_HARDWARE"
 				(path "/8bc2c25a-a1f1-4ce8-b96a-a4f8f4c35079/1e81ec4a-7813-42c9-8244-ecd5bd9e7dba/fbf84a60-b5da-4635-a9d4-00654e4ba37c"
-					(reference "R131")
+					(reference "R1302")
+					(unit 1)
+				)
+				(path "/8bc2c25a-a1f1-4ce8-b96a-a4f8f4c35079/cc03c9bc-7d6e-4340-8742-d977d081ffa4/12593d4c-79db-4c11-831b-696dda13072a"
+					(reference "R2302")
 					(unit 1)
 				)
@@
 		(in_pos_files yes)
 		(dnp no)
-		(property "Reference" "C135"
+		(property "Reference" "C1301"
 			(at 177.8 82.55 90)
 			(show_name no)
@@
 			(project "VESC6_OPEN_HARDWARE"
 				(path "/8bc2c25a-a1f1-4ce8-b96a-a4f8f4c35079/1e81ec4a-7813-42c9-8244-ecd5bd9e7dba/fbf84a60-b5da-4635-a9d4-00654e4ba37c"
-					(reference "C135")
+					(reference "C1301")
+					(unit 1)
+				)
+				(path "/8bc2c25a-a1f1-4ce8-b96a-a4f8f4c35079/cc03c9bc-7d6e-4340-8742-d977d081ffa4/12593d4c-79db-4c11-831b-696dda13072a"
+					(reference "C2301")
 					(unit 1)
 				)
@@
 		(in_pos_files yes)
 		(dnp no)
-		(property "Reference" "#PWR0114"
+		(property "Reference" "#PWR01302"
 			(at 163.83 118.11 0)
 			(hide yes)
@@
 			(project "VESC6_OPEN_HARDWARE"
 				(path "/8bc2c25a-a1f1-4ce8-b96a-a4f8f4c35079/1e81ec4a-7813-42c9-8244-ecd5bd9e7dba/fbf84a60-b5da-4635-a9d4-00654e4ba37c"
-					(reference "#PWR0114")
+					(reference "#PWR01302")
+					(unit 1)
+				)
+				(path "/8bc2c25a-a1f1-4ce8-b96a-a4f8f4c35079/cc03c9bc-7d6e-4340-8742-d977d081ffa4/12593d4c-79db-4c11-831b-696dda13072a"
+					(reference "#PWR02302")
 					(unit 1)
 				)
@@
 		(in_pos_files yes)
 		(dnp no)
-		(property "Reference" "#PWR0113"
+		(property "Reference" "#PWR01301"
 			(at 127 102.87 0)
 			(hide yes)
@@
 			(project "VESC6_OPEN_HARDWARE"
 				(path "/8bc2c25a-a1f1-4ce8-b96a-a4f8f4c35079/1e81ec4a-7813-42c9-8244-ecd5bd9e7dba/fbf84a60-b5da-4635-a9d4-00654e4ba37c"
-					(reference "#PWR0113")
+					(reference "#PWR01301")
+					(unit 1)
+				)
+				(path "/8bc2c25a-a1f1-4ce8-b96a-a4f8f4c35079/cc03c9bc-7d6e-4340-8742-d977d081ffa4/12593d4c-79db-4c11-831b-696dda13072a"
+					(reference "#PWR02301")
 					(unit 1)
 				)
@@
 		(in_pos_files yes)
 		(dnp no)
-		(property "Reference" "C136"
+		(property "Reference" "C1302"
 			(at 177.8 92.71 90)
 			(show_name no)
@@
 			(project "VESC6_OPEN_HARDWARE"
 				(path "/8bc2c25a-a1f1-4ce8-b96a-a4f8f4c35079/1e81ec4a-7813-42c9-8244-ecd5bd9e7dba/fbf84a60-b5da-4635-a9d4-00654e4ba37c"
-					(reference "C136")
+					(reference "C1302")
+					(unit 1)
+				)
+				(path "/8bc2c25a-a1f1-4ce8-b96a-a4f8f4c35079/cc03c9bc-7d6e-4340-8742-d977d081ffa4/12593d4c-79db-4c11-831b-696dda13072a"
+					(reference "C2302")
 					(unit 1)
 				)
@@
 		(in_pos_files yes)
 		(dnp no)
-		(property "Reference" "#PWR0112"
+		(property "Reference" "#PWR01303"
 			(at 184.15 87.63 0)
 			(hide yes)
@@
 			(project "VESC6_OPEN_HARDWARE"
 				(path "/8bc2c25a-a1f1-4ce8-b96a-a4f8f4c35079/1e81ec4a-7813-42c9-8244-ecd5bd9e7dba/fbf84a60-b5da-4635-a9d4-00654e4ba37c"
-					(reference "#PWR0112")
+					(reference "#PWR01303")
+					(unit 1)
+				)
+				(path "/8bc2c25a-a1f1-4ce8-b96a-a4f8f4c35079/cc03c9bc-7d6e-4340-8742-d977d081ffa4/12593d4c-79db-4c11-831b-696dda13072a"
+					(reference "#PWR02303")
 					(unit 1)
 				)
@@
 		(in_pos_files yes)
 		(dnp no)
-		(property "Reference" "R130"
+		(property "Reference" "R1301"
 			(at 113.03 87.63 90)
 			(show_name no)
@@
 			(project "VESC6_OPEN_HARDWARE"
 				(path "/8bc2c25a-a1f1-4ce8-b96a-a4f8f4c35079/1e81ec4a-7813-42c9-8244-ecd5bd9e7dba/fbf84a60-b5da-4635-a9d4-00654e4ba37c"
-					(reference "R130")
+					(reference "R1301")
+					(unit 1)
+				)
+				(path "/8bc2c25a-a1f1-4ce8-b96a-a4f8f4c35079/cc03c9bc-7d6e-4340-8742-d977d081ffa4/12593d4c-79db-4c11-831b-696dda13072a"
+					(reference "R2301")
 					(unit 1)
 				)
@@
 		(in_pos_files yes)
 		(dnp no)
-		(property "Reference" "U107"
+		(property "Reference" "U1301"
 			(at 148.59 79.5782 0)
 			(show_name no)
@@
 			(project "VESC6_OPEN_HARDWARE"
 				(path "/8bc2c25a-a1f1-4ce8-b96a-a4f8f4c35079/1e81ec4a-7813-42c9-8244-ecd5bd9e7dba/fbf84a60-b5da-4635-a9d4-00654e4ba37c"
-					(reference "U107")
-					(unit 1)
-				)
+					(reference "U1301")
+					(unit 1)
+				)
+				(path "/8bc2c25a-a1f1-4ce8-b96a-a4f8f4c35079/cc03c9bc-7d6e-4340-8742-d977d081ffa4/12593d4c-79db-4c11-831b-696dda13072a"
+					(reference "U2301")
+					(unit 1)
+				)

Commit message: finishing touches
Parts:
- C1301, C1302: LCSC (none) -> C14663; LCSC part no. C14663 -> (none); now not fitted; now left out of the parts list
- R1301, R1302: LCSC (none) -> C21190; LCSC part no. C21190 -> (none); now not fitted; now left out of the parts list
- U1301: LCSC (none) -> C967633; LCSC part no. C967633 -> (none); now not fitted; now left out of the parts list
Changed lines of the file:
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@@
 		(body_style 1)
 		(exclude_from_sim no)
-		(in_bom yes)
+		(in_bom no)
 		(on_board yes)
 		(in_pos_files yes)
-		(dnp no)
+		(dnp yes)
 		(property "Reference" "R1302"
 			(at 121.92 87.63 90)
@@
 			)
 		)
-		(property "LCSC part no." "C21190"
-			(at 124.46 87.63 0)
-			(hide yes)
-			(show_name no)
-			(do_not_autoplace no)
-			(effects
-				(font
-					(size 1.27 1.27)
-				)
-			)
-		)
 		(property "Critical" "N"
 			(at 124.46 87.63 0)
@@
 		(property "MFP" "0603WAF1001T5E"
 			(at 124.46 87.63 0)
+			(hide yes)
+			(show_name no)
+			(do_not_autoplace no)
+			(effects
+				(font
+					(size 1.27 1.27)
+				)
+			)
+		)
+		(property "LCSC" "C21190"
+			(at 124.46 87.63 90)
 			(hide yes)
 			(show_name no)
@@
 		(body_style 1)
 		(exclude_from_sim no)
-		(in_bom yes)
+		(in_bom no)
 		(on_board yes)
 		(in_pos_files yes)
-		(dnp no)
+		(dnp yes)
 		(property "Reference" "C1301"
 			(at 177.8 82.55 90)
@@
 			)
 		)
-		(property "LCSC part no." "C14663"
-			(at 176.53 83.82 0)
-			(hide yes)
-			(show_name no)
-			(do_not_autoplace no)
-			(effects
-				(font
-					(size 1.27 1.27)
-				)
-			)
-		)
 		(property "Critical" "N"
 			(at 176.53 83.82 0)
@@
 		(property "MFP" "CC0603KRX7R9BB104"
 			(at 176.53 83.82 0)
+			(hide yes)
+			(show_name no)
+			(do_not_autoplace no)
+			(effects
+				(font
+					(size 1.27 1.27)
+				)
+			)
+		)
+		(property "LCSC" "C14663"
+			(at 176.53 83.82 90)
 			(hide yes)
 			(show_name no)
@@
 		(body_style 1)
 		(exclude_from_sim no)
-		(in_bom yes)
+		(in_bom no)
 		(on_board yes)
 		(in_pos_files yes)
-		(dnp no)
+		(dnp yes)
 		(property "Reference" "C1302"
 			(at 177.8 92.71 90)
@@
 			)
 		)
-		(property "LCSC part no." "C14663"
-			(at 176.53 91.44 0)
-			(hide yes)
-			(show_name no)
-			(do_not_autoplace no)
-			(effects
-				(font
-					(size 1.27 1.27)
-				)
-			)
-		)
 		(property "Critical" "N"
 			(at 176.53 91.44 0)
@@
 		(property "MFP" "CC0603KRX7R9BB104"
 			(at 176.53 91.44 0)
+			(hide yes)
+			(show_name no)
+			(do_not_autoplace no)
+			(effects
+				(font
+					(size 1.27 1.27)
+				)
+			)
+		)
+		(property "LCSC" "C14663"
+			(at 176.53 91.44 90)
 			(hide yes)
 			(show_name no)
@@
 		(body_style 1)
 		(exclude_from_sim no)
-		(in_bom yes)
+		(in_bom no)
 		(on_board yes)
 		(in_pos_files yes)
-		(dnp no)
+		(dnp yes)
 		(property "Reference" "R1301"
 			(at 113.03 87.63 90)
@@
 			)
 		)
-		(property "LCSC part no." "C21190"
-			(at 115.57 87.63 0)
-			(hide yes)
-			(show_name no)
-			(do_not_autoplace no)
-			(effects
-				(font
-					(size 1.27 1.27)
-				)
-			)
-		)
 		(property "Critical" "N"
 			(at 115.57 87.63 0)
@@
 		(property "MFP" "0603WAF1001T5E"
 			(at 115.57 87.63 0)
+			(hide yes)
+			(show_name no)
+			(do_not_autoplace no)
+			(effects
+				(font
+					(size 1.27 1.27)
+				)
+			)
+		)
+		(property "LCSC" "C21190"
+			(at 115.57 87.63 90)
 			(hide yes)
 			(show_name no)
@@
 		(body_style 1)
 		(exclude_from_sim no)
-		(in_bom yes)
+		(in_bom no)
 		(on_board yes)
 		(in_pos_files yes)
-		(dnp no)
+		(dnp yes)
 		(property "Reference" "U1301"
 			(at 148.59 79.5782 0)
@@
 			)
 		)
-		(property "LCSC part no." "C967633"
-			(at 148.59 101.6 0)
-			(hide yes)
-			(show_name no)
-			(do_not_autoplace no)
-			(effects
-				(font
-					(size 1.27 1.27)
-				)
-			)
-		)
 		(property "Critical" "Y"
 			(at 148.59 101.6 0)
@@
 			(at 148.59 101.6 0)
 			(hide yes)
+			(show_name no)
+			(do_not_autoplace no)
+			(effects
+				(font
+					(size 1.27 1.27)
+				)
+			)
+		)
+		(property "LCSC" "C967633"
+			(at 148.59 101.6 0)
+			(hide yes)

Commit message: more tweaks
Other:
- company: (none) -> craigg96, Tomáš Kuchta
- title: (none) -> 2ch VESC based on VESC6
Changed lines of the file:
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@@
 	(paper "A4")
 	(title_block
+		(title "2ch VESC based on VESC6")
 		(date "2025-03-23")
-		(rev "A")
-		(comment 1 "Drawn By: CG")
+		(rev "B")
+		(company "craigg96, Tomáš Kuchta")
 	)
 	(junction
