File: mcu.kicad_sch (KiCad schematic)
At the start: 13 parts, among them U1 STM32F40X_LQFP64, X1 8m

Commit message: prep for chaneling. fixed the connector references, added cha to this schematic.
Connections:
- net VCC renamed +3V3a
Changed lines of the file:
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@@
 			)
 		)
-		(property "Value" "VCC"
+		(property "Value" "+3V3a"
 			(at 185.8518 87.0458 0)
 			(show_name no)
@@
 			)
 		)
-		(property "Value" "VCC"
+		(property "Value" "+3V3a"
 			(at 187.96 123.19 0)
 			(show_name no)
@@
 			)
 		)
-		(property "Value" "VCC"
+		(property "Value" "+3V3a"
 			(at 195.58 121.92 0)
 			(show_name no)
@@
 			)
 		)
-		(property "Value" "VCC"
+		(property "Value" "+3V3a"
 			(at 246.8118 38.7858 0)
 			(show_name no)

Commit message: more fixes for channels
Parts:
- renumbered C2 to C1006, C3 to C1007, C4 to C1008, C7 to C1009, C5 to C1010, C6 to C1011, C8 to C1012, C9 to C1013, C10 to C1014, C11 to C1015, C12 to C1016, U1 to U1003, X1 to X1001
Connections:
- net +3V3a renamed +3V3
Other:
- moved on the sheet: C1011, C1013, C1014, C1015, C1016

Commit message: relinked UUIDs
Parts:
- renumbered C1006 to C137, C1007 to C138, C1008 to C139, C1009 to C140, C1010 to C141, C1011 to C142, C1012 to C143, C1013 to C144, C1014 to C145, C1015 to C146, C1016 to C147, U1003 to U109, X1001 to X101
Changed lines of the file:
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@@
 		(in_pos_files yes)
 		(dnp no)
-		(property "Reference" "C1006"
+		(property "Reference" "C137"
 			(at 195.58 31.75 0)
 			(show_name no)
@@
 			(project "VESC6_OPEN_HARDWARE"
 				(path "/8bc2c25a-a1f1-4ce8-b96a-a4f8f4c35079/1e81ec4a-7813-42c9-8244-ecd5bd9e7dba/6c9ef783-93a1-4b42-9992-c17d757241d1"
-					(reference "C1006")
+					(reference "C137")
 					(unit 1)
 				)
@@
 		(in_pos_files yes)
 		(dnp no)
-		(property "Reference" "C1012"
+		(property "Reference" "C143"
 			(at 217.17 31.75 0)
 			(show_name no)
@@
 			(project "VESC6_OPEN_HARDWARE"
 				(path "/8bc2c25a-a1f1-4ce8-b96a-a4f8f4c35079/1e81ec4a-7813-42c9-8244-ecd5bd9e7dba/6c9ef783-93a1-4b42-9992-c17d757241d1"
-					(reference "C1012")
+					(reference "C143")
 					(unit 1)
 				)
@@
 		(in_pos_files yes)
 		(dnp no)
-		(property "Reference" "C1009"
+		(property "Reference" "C140"
 			(at 202.311 59.7916 0)
 			(show_name no)
@@
 			(project "VESC6_OPEN_HARDWARE"
 				(path "/8bc2c25a-a1f1-4ce8-b96a-a4f8f4c35079/1e81ec4a-7813-42c9-8244-ecd5bd9e7dba/6c9ef783-93a1-4b42-9992-c17d757241d1"
-					(reference "C1009")
+					(reference "C140")
 					(unit 1)
 				)
@@
 		(in_pos_files yes)
 		(dnp no)
-		(property "Reference" "C1010"
+		(property "Reference" "C141"
 			(at 204.47 127 0)
 			(show_name no)
@@
 			(project "VESC6_OPEN_HARDWARE"
 				(path "/8bc2c25a-a1f1-4ce8-b96a-a4f8f4c35079/1e81ec4a-7813-42c9-8244-ecd5bd9e7dba/6c9ef783-93a1-4b42-9992-c17d757241d1"
-					(reference "C1010")
+					(reference "C141")
 					(unit 1)
 				)
@@
 		(in_pos_files yes)
 		(dnp no)
-		(property "Reference" "C1011"
+		(property "Reference" "C142"
 			(at 217.17 127 0)
 			(show_name no)
@@
 			(project "VESC6_OPEN_HARDWARE"
 				(path "/8bc2c25a-a1f1-4ce8-b96a-a4f8f4c35079/1e81ec4a-7813-42c9-8244-ecd5bd9e7dba/6c9ef783-93a1-4b42-9992-c17d757241d1"
-					(reference "C1011")
+					(reference "C142")
 					(unit 1)
 				)
@@
 		(in_pos_files yes)
 		(dnp no)
-		(property "Reference" "C1007"
+		(property "Reference" "C138"
 			(at 198.12 136.398 90)
 			(show_name no)
@@
 			(project "VESC6_OPEN_HARDWARE"
 				(path "/8bc2c25a-a1f1-4ce8-b96a-a4f8f4c35079/1e81ec4a-7813-42c9-8244-ecd5bd9e7dba/6c9ef783-93a1-4b42-9992-c17d757241d1"
-					(reference "C1007")
+					(reference "C138")
 					(unit 1)
 				)
@@
 		(in_pos_files yes)
 		(dnp no)
-		(property "Reference" "C1008"
+		(property "Reference" "C139"
 			(at 198.12 149.606 90)
 			(show_name no)
@@
 			(project "VESC6_OPEN_HARDWARE"
 				(path "/8bc2c25a-a1f1-4ce8-b96a-a4f8f4c35079/1e81ec4a-7813-42c9-8244-ecd5bd9e7dba/6c9ef783-93a1-4b42-9992-c17d757241d1"
-					(reference "C1008")
+					(reference "C139")
 					(unit 1)
 				)
@@
 		(in_pos_files yes)
 		(dnp no)
-		(property "Reference" "U1003"
+		(property "Reference" "U109"
 			(at 153.67 24.4602 0)
 			(show_name no)
@@
 			(project "VESC6_OPEN_HARDWARE"
 				(path "/8bc2c25a-a1f1-4ce8-b96a-a4f8f4c35079/1e81ec4a-7813-42c9-8244-ecd5bd9e7dba/6c9ef783-93a1-4b42-9992-c17d757241d1"
-					(reference "U1003")
+					(reference "U109")
 					(unit 1)
 				)
@@
 		(in_pos_files yes)
 		(dnp no)
-		(property "Reference" "X1001"
+		(property "Reference" "X101"
 			(at 205.74 34.29 0)
 			(show_name no)
@@
 			(project "VESC6_OPEN_HARDWARE"
 				(path "/8bc2c25a-a1f1-4ce8-b96a-a4f8f4c35079/1e81ec4a-7813-42c9-8244-ecd5bd9e7dba/6c9ef783-93a1-4b42-9992-c17d757241d1"
-					(reference "X1001")
+					(reference "X101")
 					(unit 1)
 				)
@@
 		(in_pos_files yes)
 		(dnp no)
-		(property "Reference" "C1013"
+		(property "Reference" "C144"
 			(at 228.6 97.79 0)
 			(show_name no)
@@
 			(project "VESC6_OPEN_HARDWARE"
 				(path "/8bc2c25a-a1f1-4ce8-b96a-a4f8f4c35079/1e81ec4a-7813-42c9-8244-ecd5bd9e7dba/6c9ef783-93a1-4b42-9992-c17d757241d1"
-					(reference "C1013")
+					(reference "C144")
 					(unit 1)
 				)
@@
 		(in_pos_files yes)
 		(dnp no)
-		(property "Reference" "C1014"
+		(property "Reference" "C145"
 			(at 238.76 97.79 0)
 			(show_name no)
@@
 			(project "VESC6_OPEN_HARDWARE"
 				(path "/8bc2c25a-a1f1-4ce8-b96a-a4f8f4c35079/1e81ec4a-7813-42c9-8244-ecd5bd9e7dba/6c9ef783-93a1-4b42-9992-c17d757241d1"
-					(reference "C1014")
+					(reference "C145")
 					(unit 1)
 				)
@@
 		(in_pos_files yes)
 		(dnp no)
-		(property "Reference" "C1015"
+		(property "Reference" "C146"
 			(at 248.92 97.79 0)
 			(show_name no)
@@
 			(project "VESC6_OPEN_HARDWARE"
 				(path "/8bc2c25a-a1f1-4ce8-b96a-a4f8f4c35079/1e81ec4a-7813-42c9-8244-ecd5bd9e7dba/6c9ef783-93a1-4b42-9992-c17d757241d1"
-					(reference "C1015")
+					(reference "C146")
 					(unit 1)
 				)
@@
 		(in_pos_files yes)
 		(dnp no)
-		(property "Reference" "C1016"
+		(property "Reference" "C147"
 			(at 259.08 97.79 0)
 			(show_name no)
@@
 			(project "VESC6_OPEN_HARDWARE"
 				(path "/8bc2c25a-a1f1-4ce8-b96a-a4f8f4c35079/1e81ec4a-7813-42c9-8244-ecd5bd9e7dba/6c9ef783-93a1-4b42-9992-c17d757241d1"
-					(reference "C1016")
+					(reference "C147")
 					(unit 1)
 				)

Commit message: it seems to work. yay
Parts:
- renumbered C137 to C1501, C138 to C1502, C139 to C1503, C140 to C1504, C141 to C1505, C142 to C1506, C143 to C1507, C144 to C1508, C145 to C1509, C146 to C1510, C147 to C1511, U109 to U1501, X101 to X1501

Commit message: finishing touches
Parts:
- C1501, C1507: LCSC (none) -> C1644; LCSC part no. C1644 -> (none)
- C1502, C1503, C1505, C1506, C1508, C1509, C1510, C1511: LCSC (none) -> C23630; LCSC part no. C23630 -> (none)
- C1504: LCSC (none) -> C14663; LCSC part no. C14663 -> (none)
- U1501: LCSC (none) -> C15742; LCSC part no. C15742 -> (none)
- X1501: LCSC (none) -> C115962; LCSC part no. C115962 -> (none)
Changed lines of the file:
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@@
-			)
-		)
-		(property "LCSC part no." "C1644"
-			(at 195.58 34.29 0)
-			(hide yes)
-			(show_name no)
-			(do_not_autoplace no)
-			(effects
-				(font
-					(size 1.27 1.27)
-				)
 			)
 		)
@@
 		)
 		(property "MFP" "CL10C150JB8NNNC"
+			(at 195.58 34.29 0)
+			(hide yes)
+			(show_name no)
+			(do_not_autoplace no)
+			(effects
+				(font
+					(size 1.27 1.27)
+				)
+			)
+		)
+		(property "LCSC" "C1644"
 			(at 195.58 34.29 0)
 			(hide yes)
@@
 			)
 		)
-		(property "LCSC part no." "C1644"
-			(at 215.9 34.29 0)
-			(hide yes)
-			(show_name no)
-			(do_not_autoplace no)
-			(effects
-				(font
-					(size 1.27 1.27)
-				)
-			)
-		)
 		(property "Critical" "N"
 			(at 215.9 34.29 0)
@@
 		)
 		(property "MFP" "CL10C150JB8NNNC"
+			(at 215.9 34.29 0)
+			(hide yes)
+			(show_name no)
+			(do_not_autoplace no)
+			(effects
+				(font
+					(size 1.27 1.27)
+				)
+			)
+		)
+		(property "LCSC" "C1644"
 			(at 215.9 34.29 0)
 			(hide yes)
@@
 			)
 		)
-		(property "LCSC part no." "C14663"
-			(at 199.39 60.96 0)
-			(hide yes)
-			(show_name no)
-			(do_not_autoplace no)
-			(effects
-				(font
-					(size 1.27 1.27)
-				)
-			)
-		)
 		(property "Critical" "N"
 			(at 199.39 60.96 0)
@@
 		)
 		(property "MFP" "CC0603KRX7R9BB104"
+			(at 199.39 60.96 0)
+			(hide yes)
+			(show_name no)
+			(do_not_autoplace no)
+			(effects
+				(font
+					(size 1.27 1.27)
+				)
+			)
+		)
+		(property "LCSC" "C14663"
 			(at 199.39 60.96 0)
 			(hide yes)
@@
 			)
 		)
-		(property "LCSC part no." "C23630"
-			(at 201.93 129.54 0)
-			(hide yes)
-			(show_name no)
-			(do_not_autoplace no)
-			(effects
-				(font
-					(size 1.27 1.27)
-				)
-			)
-		)
 		(property "Critical" "N"
 			(at 201.93 129.54 0)
@@
 		)
 		(property "MFP" "CL10A225KO8NNNC"
+			(at 201.93 129.54 0)
+			(hide yes)
+			(show_name no)
+			(do_not_autoplace no)
+			(effects
+				(font
+					(size 1.27 1.27)
+				)
+			)
+		)
+		(property "LCSC" "C23630"
 			(at 201.93 129.54 0)
 			(hide yes)
@@
 			)
 		)
-		(property "LCSC part no." "C23630"
-			(at 214.63 129.54 0)
-			(hide yes)
-			(show_name no)
-			(do_not_autoplace no)
-			(effects
-				(font
-					(size 1.27 1.27)
-				)
-			)
-		)
 		(property "Critical" "N"
 			(at 214.63 129.54 0)
@@
 		)
 		(property "MFP" "CL10A225KO8NNNC"
+			(at 214.63 129.54 0)
+			(hide yes)
+			(show_name no)
+			(do_not_autoplace no)
+			(effects
+				(font
+					(size 1.27 1.27)
+				)
+			)
+		)
+		(property "LCSC" "C23630"
 			(at 214.63 129.54 0)
 			(hide yes)
@@
 			)
 		)
-		(property "LCSC part no." "C23630"
-			(at 198.12 139.7 0)
-			(hide yes)
-			(show_name no)
-			(do_not_autoplace no)
-			(effects
-				(font
-					(size 1.27 1.27)
-				)
-			)
-		)
 		(property "Critical" "N"
 			(at 198.12 139.7 0)
@@
 		(property "MFP" "CL10A225KO8NNNC"
 			(at 198.12 139.7 0)
+			(hide yes)
+			(show_name no)
+			(do_not_autoplace no)
+			(effects
+				(font
+					(size 1.27 1.27)
+				)
+			)
+		)
+		(property "LCSC" "C23630"
+			(at 198.12 139.7 90)
 			(hide yes)
 			(show_name no)
@@
 			)
 		)
-		(property "LCSC part no." "C23630"
-			(at 198.12 146.05 0)
-			(hide yes)
-			(show_name no)
-			(do_not_autoplace no)
-			(effects
-				(font
-					(size 1.27 1.27)
-				)
-			)
-		)
 		(property "Critical" "N"
 			(at 198.12 146.05 0)
@@
 		(property "MFP" "CL10A225KO8NNNC"
 			(at 198.12 146.05 0)
+			(hide yes)
+			(show_name no)
+			(do_not_autoplace no)
+			(effects
+				(font
+					(size 1.27 1.27)
+				)
+			)
+		)
+		(property "LCSC" "C23630"
+			(at 198.12 146.05 90)
 			(hide yes)
 			(show_name no)
@@
 			)
 		)
-		(property "LCSC part no." "C15742"
-			(at 153.67 86.36 0)
-			(hide yes)
-			(show_name no)
-			(do_not_autoplace no)
-			(effects
-				(font
-					(size 1.27 1.27)
-				)
-			)
-		)
 		(property "Critical" "Y"
 			(at 153.67 86.36 0)
@@
 		)
 		(property "MFP" "STM32F405RGT6"
+			(at 153.67 86.36 0)
+			(hide yes)
+			(show_name no)
+			(do_not_autoplace no)
+			(effects
+				(font
+					(size 1.27 1.27)
+				)
+			)
+		)
+		(property "LCSC" "C15742"
 			(at 153.67 86.36 0)
 			(hide yes)
@@
 			)
 		)
-		(property "LCSC part no." "C115962"
-			(at 205.74 38.1 0)
-			(hide yes)
-			(show_name no)
-			(do_not_autoplace no)
-			(effects
-				(font
-					(size 1.27 1.27)
-				)
-			)
-		)
 		(property "MFP" "X50328MSB2GI"
 			(at 205.74 38.1 0)
@@
 		)
 		(property "Link" "https://jlcpcb.com/partdetail/YangxingTech-X50328MSB2GI/C115962"
+			(at 205.74 38.1 0)
+			(hide yes)
+			(show_name no)
+			(do_not_autoplace no)
+			(effects
+				(font
+					(size 1.27 1.27)
+				)
+			)
+		)
+		(property "LCSC" "C115962"
 			(at 205.74 38.1 0)
 			(hide yes)
@@
 			)
 		)
-		(property "LCSC part no." "C23630"
-			(at 227.33 100.33 0)
-			(hide yes)
-			(show_name no)
-			(do_not_autoplace no)
-			(effects
-				(font
-					(size 1.27 1.27)
-				)
-			)
-		)
 		(property "Critical" "N"
 			(at 227.33 100.33 0)
@@
 		)
 		(property "MFP" "CL10A225KO8NNNC"
+			(at 227.33 100.33 0)
+			(hide yes)
+			(show_name no)
+			(do_not_autoplace no)
+			(effects
+				(font
+					(size 1.27 1.27)
+				)
+			)
+		)
+		(property "LCSC" "C23630"
 			(at 227.33 100.33 0)
 			(hide yes)
@@
 			)
 		)
-		(property "LCSC part no." "C23630"
-			(at 237.49 100.33 0)
-			(hide yes)
-			(show_name no)
-			(do_not_autoplace no)
-			(effects
-				(font
-					(size 1.27 1.27)
-				)
-			)
-		)
 		(property "Critical" "N"
 			(at 237.49 100.33 0)
@@
 		)
 		(property "MFP" "CL10A225KO8NNNC"
+			(at 237.49 100.33 0)
+			(hide yes)
+			(show_name no)
+			(do_not_autoplace no)
+			(effects
+				(font
+					(size 1.27 1.27)
+				)
+			)
+		)
+		(property "LCSC" "C23630"
 			(at 237.49 100.33 0)
 			(hide yes)
@@
 			)
 		)
-		(property "LCSC part no." "C23630"
-			(at 247.65 100.33 0)
-			(hide yes)
-			(show_name no)
-			(do_not_autoplace no)
-			(effects
-				(font
-					(size 1.27 1.27)
-				)
-			)
-		)
 		(property "Critical" "N"
 			(at 247.65 100.33 0)
@@
 		)
 		(property "MFP" "CL10A225KO8NNNC"
+			(at 247.65 100.33 0)
+			(hide yes)
+			(show_name no)
+			(do_not_autoplace no)
+			(effects
+				(font
+					(size 1.27 1.27)
+				)
+			)
+		)
+		(property "LCSC" "C23630"
 			(at 247.65 100.33 0)
 			(hide yes)
@@
 			)
 		)
-		(property "LCSC part no." "C23630"
-			(at 257.81 100.33 0)
-			(hide yes)
-			(show_name no)
-			(do_not_autoplace no)
-			(effects
-				(font
-					(size 1.27 1.27)
-				)
-			)
-		)
 		(property "Critical" "N"
 			(at 257.81 100.33 0)
@@
 			(at 257.81 100.33 0)
 			(hide yes)
+			(show_name no)
+			(do_not_autoplace no)
+			(effects
+				(font
+					(size 1.27 1.27)
+				)
+			)
+		)
+		(property "LCSC" "C23630"
+			(at 257.81 100.33 0)
+			(hide yes)

Commit message: more tweaks
Other:
- company: (none) -> craigg96, Tomáš Kuchta
- title: (none) -> 2ch VESC based on VESC6
Changed lines of the file:
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@@
 	(paper "A4")
 	(title_block
+		(title "2ch VESC based on VESC6")
 		(date "2025-03-23")
-		(rev "A")
-		(comment 1 "Drawn By: CG")
+		(rev "B")
+		(company "craigg96, Tomáš Kuchta")
 	)
 	(text "Bypass, place next to VDD pins"
