File: power.kicad_sch (KiCad schematic)
At the start: 45 parts, among them P10 PH_A, P11 SUPPLY, P12 GND, P8 PH_C, P9 PH_B, Q1 STL130N6F7, Q2 STL130N6F7, Q3 STL130N6F7, Q4 STL130N6F7, Q5 STL130N6F7, Q6 STL130N6F7, U5 AD8418, U6 AD8418, U7 AD8418

Commit message: prep for chaneling. fixed the connector references, added cha to this schematic.
Connections:
- net VCC renamed +3V3a
Changed lines of the file:
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@@
 			)
 		)
-		(property "Value" "VCC"
+		(property "Value" "+3V3a"
 			(at 140.1318 67.9958 0)
 			(show_name no)
@@
 			)
 		)
-		(property "Value" "VCC"
+		(property "Value" "+3V3a"
 			(at 46.1518 69.2658 0)
 			(show_name no)
@@
 			)
 		)
-		(property "Value" "VCC"
+		(property "Value" "+3V3a"
 			(at 227.7618 69.2658 0)
 			(show_name no)
@@
 			)
 		)
-		(property "Value" "VCC"
+		(property "Value" "+3V3a"
 			(at 142.6718 128.9558 0)
 			(show_name no)

Commit message: more fixes for channels
Parts:
- removed C29, C30, C45: 4.7n, Capacitor_SMD:C_0603_1608Metric, symbol Device:C
- removed C35, C36, C38, C42: 2.2uF, Capacitor_SMD:C_0603_1608Metric, symbol Device:C
- removed C37, C39, C40, C41, C43, C44: 4.7u_100v, Capacitor_SMD:C_1210_3225Metric, symbol Device:C
- removed C48, C49, C50, C51: 220u_63v, Capacitor_SMD:CP_Elec_10x10.5, symbol Device:C
- removed P10: PH_A, Connector_Pin:Pin_D1.3mm_L11.0mm_LooseFit, symbol Connector_Generic:Conn_01x01
- removed P11: SUPPLY, Connector_Pin:Pin_D1.3mm_L11.0mm_LooseFit, symbol Connector_Generic:Conn_01x01
- removed P12: GND, Connector_Pin:Pin_D1.3mm_L11.0mm_LooseFit, symbol Connector_Generic:Conn_01x01
- removed P8: PH_C, Connector_Pin:Pin_D1.3mm_L11.0mm_LooseFit, symbol Connector_Generic:Conn_01x01
- removed P9: PH_B, Connector_Pin:Pin_D1.3mm_L11.0mm_LooseFit, symbol Connector_Generic:Conn_01x01
- removed Q1, Q2, Q3, Q4, Q5, Q6: STL130N6F7, CustomFootprints:NVMFS5C612NL, symbol bldc:IRF7749L1PBF
- removed R24, R29, R32: 0.0005R, CustomFootprints:2512_SHUNT, symbol Device:R
- removed R25, R26, R30, R31, R33, R34: 4.7R, Resistor_SMD:R_0603_1608Metric, symbol Device:R
- removed R27: NTC 10k, Resistor_SMD:R_0603_1608Metric, symbol Device:R
- removed R28: 10k, Resistor_SMD:R_0603_1608Metric, symbol Device:R
- removed R35, R36, R37: 100R, Resistor_SMD:R_0603_1608Metric, symbol Device:R
- removed U5, U6, U7: AD8418, Package_SO:SOIC-8_3.9x4.9mm_P1.27mm, symbol Amplifier_Current:AD8418
- added C1047, C1048, C1049, C1050: 220u_63v, Capacitor_SMD:CP_Elec_10x10.5, symbol Device:C
- added P1009: SUPPLY, Connector_Pin:Pin_D1.3mm_L11.0mm_LooseFit, symbol Connector_Generic:Conn_01x01
- added P1010: GND, Connector_Pin:Pin_D1.3mm_L11.0mm_LooseFit, symbol Connector_Generic:Conn_01x01
Connections:
- net GND: now also C1047.2, C1048.2, C1049.2, C1050.2, P1010.1 (Pin_1)
- net SUPPLY: now also C1047.1, C1048.1, C1049.1, C1050.1, P1009.1 (Pin_1)

Commit message: relinked UUIDs
Parts:
- renumbered C1047 to C1, C1048 to C2, C1049 to C3, C1050 to C4, P1009 to P1, P1010 to P2
Changed lines of the file:
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@@
 		(in_pos_files yes)
 		(dnp no)
-		(property "Reference" "P1010"
+		(property "Reference" "P2"
 			(at 182.88 100.33 0)
 			(show_name no)
@@
 			(project "VESC6_OPEN_HARDWARE"
 				(path "/8bc2c25a-a1f1-4ce8-b96a-a4f8f4c35079/bb515b26-eb2d-4e36-ac67-211043564e95"
-					(reference "P1010")
+					(reference "P2")
 					(unit 1)
 				)
@@
 		(in_pos_files yes)
 		(dnp no)
-		(property "Reference" "C1048"
+		(property "Reference" "C2"
 			(at 135.89 91.44 0)
 			(show_name no)
@@
 			(project "VESC6_OPEN_HARDWARE"
 				(path "/8bc2c25a-a1f1-4ce8-b96a-a4f8f4c35079/bb515b26-eb2d-4e36-ac67-211043564e95"
-					(reference "C1048")
+					(reference "C2")
 					(unit 1)
 				)
@@
 		(in_pos_files yes)
 		(dnp no)
-		(property "Reference" "C1049"
+		(property "Reference" "C3"
 			(at 147.32 91.44 0)
 			(show_name no)
@@
 			(project "VESC6_OPEN_HARDWARE"
 				(path "/8bc2c25a-a1f1-4ce8-b96a-a4f8f4c35079/bb515b26-eb2d-4e36-ac67-211043564e95"
-					(reference "C1049")
+					(reference "C3")
 					(unit 1)
 				)
@@
 		(in_pos_files yes)
 		(dnp no)
-		(property "Reference" "C1047"
+		(property "Reference" "C1"
 			(at 123.19 91.44 0)
 			(show_name no)
@@
 			(project "VESC6_OPEN_HARDWARE"
 				(path "/8bc2c25a-a1f1-4ce8-b96a-a4f8f4c35079/bb515b26-eb2d-4e36-ac67-211043564e95"
-					(reference "C1047")
+					(reference "C1")
 					(unit 1)
 				)
@@
 		(in_pos_files yes)
 		(dnp no)
-		(property "Reference" "C1050"
+		(property "Reference" "C4"
 			(at 160.02 91.44 0)
 			(show_name no)
@@
 			(project "VESC6_OPEN_HARDWARE"
 				(path "/8bc2c25a-a1f1-4ce8-b96a-a4f8f4c35079/bb515b26-eb2d-4e36-ac67-211043564e95"
-					(reference "C1050")
+					(reference "C4")
 					(unit 1)
 				)
@@
 		(in_pos_files yes)
 		(dnp no)
-		(property "Reference" "P1009"
+		(property "Reference" "P1"
 			(at 182.88 80.01 0)
 			(show_name no)
@@
 			(project "VESC6_OPEN_HARDWARE"
 				(path "/8bc2c25a-a1f1-4ce8-b96a-a4f8f4c35079/bb515b26-eb2d-4e36-ac67-211043564e95"
-					(reference "P1009")
+					(reference "P1")
 					(unit 1)
 				)

Commit message: it seems to work. yay
Parts:
- renumbered C1 to C201, C2 to C202, C3 to C203, C4 to C204, P1 to P201, P2 to P202
Changed lines of the file:
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@@
 		(dnp no)
 		(fields_autoplaced yes)
-		(property "Reference" "#FLG01001"
+		(property "Reference" "#FLG0202"
 			(at 173.99 107.315 0)
 			(hide yes)
@@
 			(project "VESC6_OPEN_HARDWARE"
 				(path "/8bc2c25a-a1f1-4ce8-b96a-a4f8f4c35079/bb515b26-eb2d-4e36-ac67-211043564e95"
-					(reference "#FLG01001")
+					(reference "#FLG0202")
 					(unit 1)
 				)
@@
 		(dnp no)
 		(fields_autoplaced yes)
-		(property "Reference" "#PWR01019"
+		(property "Reference" "#PWR0201"
 			(at 158.75 81.28 0)
 			(hide yes)
@@
 			(project "VESC6_OPEN_HARDWARE"
 				(path "/8bc2c25a-a1f1-4ce8-b96a-a4f8f4c35079/bb515b26-eb2d-4e36-ac67-211043564e95"
-					(reference "#PWR01019")
+					(reference "#PWR0201")
 					(unit 1)
 				)
@@
 		(in_pos_files yes)
 		(dnp no)
-		(property "Reference" "P2"
+		(property "Reference" "P202"
 			(at 182.88 100.33 0)
 			(show_name no)
@@
 			(project "VESC6_OPEN_HARDWARE"
 				(path "/8bc2c25a-a1f1-4ce8-b96a-a4f8f4c35079/bb515b26-eb2d-4e36-ac67-211043564e95"
-					(reference "P2")
+					(reference "P202")
 					(unit 1)
 				)
@@
 		(in_pos_files yes)
 		(dnp no)
-		(property "Reference" "#PWR070"
+		(property "Reference" "#PWR0202"
 			(at 158.75 115.57 0)
 			(hide yes)
@@
 			(project "VESC6_OPEN_HARDWARE"
 				(path "/8bc2c25a-a1f1-4ce8-b96a-a4f8f4c35079/bb515b26-eb2d-4e36-ac67-211043564e95"
-					(reference "#PWR070")
+					(reference "#PWR0202")
 					(unit 1)
 				)
@@
 		(dnp no)
 		(fields_autoplaced yes)
-		(property "Reference" "#FLG01002"
+		(property "Reference" "#FLG0201"
 			(at 173.99 78.105 0)
 			(hide yes)
@@
 			(project "VESC6_OPEN_HARDWARE"
 				(path "/8bc2c25a-a1f1-4ce8-b96a-a4f8f4c35079/bb515b26-eb2d-4e36-ac67-211043564e95"
-					(reference "#FLG01002")
+					(reference "#FLG0201")
 					(unit 1)
 				)
@@
 		(in_pos_files yes)
 		(dnp no)
-		(property "Reference" "C2"
+		(property "Reference" "C202"
 			(at 135.89 91.44 0)
 			(show_name no)
@@
 			(project "VESC6_OPEN_HARDWARE"
 				(path "/8bc2c25a-a1f1-4ce8-b96a-a4f8f4c35079/bb515b26-eb2d-4e36-ac67-211043564e95"
-					(reference "C2")
+					(reference "C202")
 					(unit 1)
 				)
@@
 		(in_pos_files yes)
 		(dnp no)
-		(property "Reference" "C3"
+		(property "Reference" "C203"
 			(at 147.32 91.44 0)
 			(show_name no)
@@
 			(project "VESC6_OPEN_HARDWARE"
 				(path "/8bc2c25a-a1f1-4ce8-b96a-a4f8f4c35079/bb515b26-eb2d-4e36-ac67-211043564e95"
-					(reference "C3")
+					(reference "C203")
 					(unit 1)
 				)
@@
 		(in_pos_files yes)
 		(dnp no)
-		(property "Reference" "C1"
+		(property "Reference" "C201"
 			(at 123.19 91.44 0)
 			(show_name no)
@@
 			(project "VESC6_OPEN_HARDWARE"
 				(path "/8bc2c25a-a1f1-4ce8-b96a-a4f8f4c35079/bb515b26-eb2d-4e36-ac67-211043564e95"
-					(reference "C1")
+					(reference "C201")
 					(unit 1)
 				)
@@
 		(in_pos_files yes)
 		(dnp no)
-		(property "Reference" "C4"
+		(property "Reference" "C204"
 			(at 160.02 91.44 0)
 			(show_name no)
@@
 			(project "VESC6_OPEN_HARDWARE"
 				(path "/8bc2c25a-a1f1-4ce8-b96a-a4f8f4c35079/bb515b26-eb2d-4e36-ac67-211043564e95"
-					(reference "C4")
+					(reference "C204")
 					(unit 1)
 				)
@@
 		(in_pos_files yes)
 		(dnp no)
-		(property "Reference" "P1"
+		(property "Reference" "P201"
 			(at 182.88 80.01 0)
 			(show_name no)
@@
 			(project "VESC6_OPEN_HARDWARE"
 				(path "/8bc2c25a-a1f1-4ce8-b96a-a4f8f4c35079/bb515b26-eb2d-4e36-ac67-211043564e95"
-					(reference "P1")
+					(reference "P201")
 					(unit 1)
 				)

Commit message: small improvements.
Parts:
- added C205: 220u_63v, Capacitor_SMD:CP_Elec_10x10.5, symbol Device:C
- added C206, C207: 4.7u_100v, Capacitor_SMD:C_1210_3225Metric, symbol Device:C
Connections:
- net GND: now also C205.2, C206.2, C207.2
- net SUPPLY: now also C205.1, C206.1, C207.1
Other:
- moved on the sheet: C201, C202, C203, C204, P201, P202

Commit message: finishing touches
Parts:
- C201, C202, C203, C204, C205: LCSC (none) -> C7471900; LCSC part no. C7471900 -> (none)
- C206, C207: LCSC (none) -> C385987; LCSC part no. C385987 -> (none)
- P201, P202: LCSC (none) -> C7200700; LCSC part no. C7200700 -> (none)
Changed lines of the file:
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@@
-			)
-		)
-		(property "LCSC part no." "C385987"
-			(at 179.07 95.25 0)
-			(hide yes)
-			(show_name no)
-			(do_not_autoplace no)
-			(effects
-				(font
-					(size 1.27 1.27)
-				)
 			)
 		)
@@
 		(property "Critical" "N"
 			(at 179.07 95.25 0)
+			(hide yes)
+			(show_name no)
+			(do_not_autoplace no)
+			(effects
+				(font
+					(size 1.27 1.27)
+				)
+			)
+		)
+		(property "LCSC" "C385987"
+			(at 179.07 95.25 90)
 			(hide yes)
 			(show_name no)
@@
 			)
 		)
-		(property "LCSC part no." "C7471900"
-			(at 163.83 95.25 0)
-			(hide yes)
-			(show_name no)
-			(do_not_autoplace no)
-			(effects
-				(font
-					(size 1.27 1.27)
-				)
-			)
-		)
 		(property "Critical" "N"
 			(at 163.83 95.25 0)
@@
 		)
 		(property "MFP" ""
+			(at 163.83 95.25 0)
+			(hide yes)
+			(show_name no)
+			(do_not_autoplace no)
+			(effects
+				(font
+					(size 1.27 1.27)
+				)
+			)
+		)
+		(property "LCSC" "C7471900"
 			(at 163.83 95.25 0)
 			(hide yes)
@@
 			)
 		)
-		(property "LCSC part no." "C7200700 "
+		(property "LCSC" "C7200700 "
 			(at 77.47 102.87 0)
 			(hide yes)
@@
 			)
 		)
-		(property "LCSC part no." "C7471900"
-			(at 114.3 93.98 0)
-			(hide yes)
-			(show_name no)
-			(do_not_autoplace no)
-			(effects
-				(font
-					(size 1.27 1.27)
-				)
-			)
-		)
 		(property "Critical" "N"
 			(at 114.3 93.98 0)
@@
 		)
 		(property "MFP" ""
+			(at 114.3 93.98 0)
+			(hide yes)
+			(show_name no)
+			(do_not_autoplace no)
+			(effects
+				(font
+					(size 1.27 1.27)
+				)
+			)
+		)
+		(property "LCSC" "C7471900"
 			(at 114.3 93.98 0)
 			(hide yes)
@@
 			)
 		)
-		(property "LCSC part no." "C7471900"
-			(at 125.73 93.98 0)
-			(hide yes)
-			(show_name no)
-			(do_not_autoplace no)
-			(effects
-				(font
-					(size 1.27 1.27)
-				)
-			)
-		)
 		(property "Critical" "N"
 			(at 125.73 93.98 0)
@@
 		)
 		(property "MFP" ""
+			(at 125.73 93.98 0)
+			(hide yes)
+			(show_name no)
+			(do_not_autoplace no)
+			(effects
+				(font
+					(size 1.27 1.27)
+				)
+			)
+		)
+		(property "LCSC" "C7471900"
 			(at 125.73 93.98 0)
 			(hide yes)
@@
 			)
 		)
-		(property "LCSC part no." "C7471900"
-			(at 101.6 93.98 0)
-			(hide yes)
-			(show_name no)
-			(do_not_autoplace no)
-			(effects
-				(font
-					(size 1.27 1.27)
-				)
-			)
-		)
 		(property "Critical" "N"
 			(at 101.6 93.98 0)
@@
 		)
 		(property "MFP" ""
+			(at 101.6 93.98 0)
+			(hide yes)
+			(show_name no)
+			(do_not_autoplace no)
+			(effects
+				(font
+					(size 1.27 1.27)
+				)
+			)
+		)
+		(property "LCSC" "C7471900"
 			(at 101.6 93.98 0)
 			(hide yes)
@@
 			)
 		)
-		(property "LCSC part no." "C385987"
-			(at 186.69 95.25 0)
-			(hide yes)
-			(show_name no)
-			(do_not_autoplace no)
-			(effects
-				(font
-					(size 1.27 1.27)
-				)
-			)
-		)
 		(property "Link" ""
 			(at 186.69 95.25 0)
@@
 		(property "Critical" "N"
 			(at 186.69 95.25 0)
+			(hide yes)
+			(show_name no)
+			(do_not_autoplace no)
+			(effects
+				(font
+					(size 1.27 1.27)
+				)
+			)
+		)
+		(property "LCSC" "C385987"
+			(at 186.69 95.25 90)
 			(hide yes)
 			(show_name no)
@@
 			)
 		)
-		(property "LCSC part no." "C7471900"
-			(at 138.43 93.98 0)
-			(hide yes)
-			(show_name no)
-			(do_not_autoplace no)
-			(effects
-				(font
-					(size 1.27 1.27)
-				)
-			)
-		)
 		(property "Critical" "N"
 			(at 138.43 93.98 0)
@@
 		)
 		(property "MFP" ""
+			(at 138.43 93.98 0)
+			(hide yes)
+			(show_name no)
+			(do_not_autoplace no)
+			(effects
+				(font
+					(size 1.27 1.27)
+				)
+			)
+		)
+		(property "LCSC" "C7471900"
 			(at 138.43 93.98 0)
 			(hide yes)
@@
 			)
 		)
-		(property "LCSC part no." "C7200700 "
+		(property "LCSC" "C7200700 "
 			(at 77.47 82.55 0)
 			(hide yes)

Commit message: more tweaks
Other:
- company: (none) -> craigg96, Tomáš Kuchta
- title: (none) -> 2ch VESC based on VESC6
Changed lines of the file:
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@@
 	(paper "A4")
 	(title_block
-		(rev "A")
+		(title "2ch VESC based on VESC6")
+		(rev "B")
+		(company "craigg96, Tomáš Kuchta")
 	)
 	(junction
